File: Romashka EC/Romashka EC.kicad_sch (KiCad schematic)
At the start: 0 parts

Commit message: 19.04.2026: setup
Parts:
- added BOOT_SW1, RESET_SW1: Omron b3u, Button_Switch_SMD:SW_SPST_B3U-1000P, symbol Switch:SW_DPST_x2
- added C1, C16, C18: 10uF, Capacitor_SMD:C_0805_2012Metric, symbol Device:C_Small
- added C10, C9: 15pF, Capacitor_SMD:C_0402_1005Metric, symbol Device:C_Small
- added C11, C12, C13, C14: 220pF, Capacitor_SMD:C_0603_1608Metric, symbol Device:C_Small
- added C15, C17, C8: 1uF, Capacitor_SMD:C_0603_1608Metric, symbol Device:C_Small
- added C19, C2, C3, C4, C5, C6, C7: 100nF, Capacitor_SMD:C_0402_1005Metric, symbol Device:C_Small
- added F1: 500mA, Fuse:Fuse_0603_1608Metric, symbol Device:Polyfuse_Small
- added J1: USB_C_Receptacle_USB2.0_16P, Connector_USB:USB_C_Receptacle_GCT_USB4105-xx-A_16P_TopMnt_Horizontal, symbol Connector:USB_C_Receptacle_USB2.0_16P
- added J2: JSB USB, Connector_JST:JST_SH_SM04B-SRSS-TB_1x04-1MP_P1.00mm_Horizontal, symbol Connector_Generic:Conn_01x04
- added J3: SOICbite, Kicad footprints:SOICbite_footprint, symbol Connector_Generic:Conn_01x08
- added R1, R2: 5.1k, Resistor_SMD:R_0603_1608Metric, symbol Device:R_Small
- added R10, R3, R4, R5, R6, R7, R8, R9: 330R, Resistor_SMD:R_0603_1608Metric, symbol Device:R_Small
- added R11: 10R, Resistor_SMD:R_0603_1608Metric, symbol Device:R_Small
- added R12: 33k, Resistor_SMD:R_0603_1608Metric, symbol Device:R_Small
- added U1: STM32G474CBTx, Package_QFP:LQFP-48_7x7mm_P0.5mm, symbol MCU_ST_STM32G4:STM32G474CBTx
- added U2: USBLC6-2P6, Package_TO_SOT_SMD:SOT-563, symbol Power_Protection:USBLC6-2P6
- added U3: TPS7A2033, Package_TO_SOT_SMD:SOT-23-5, symbol Regulator_Linear:TLV75533PDBV
- added Y1: 8Mhz 12pF, Crystal:Crystal_SMD_3225-4Pin_3.2x2.5mm, symbol Device:Crystal_GND24_Small
Connections:
- new net: R8.2, U1.15 (PA7)
- new net: C10.2, U1.6 (PF1), Y1.1
- new net: C9.2, U1.5 (PF0), Y1.3
- new net: J1.B5 (CC2), R2.1
- new net: R9.2, U1.16 (PB0)
- new net: C14.1, R6.1, U1.31 (PA9)
- new net: R10.2, U1.17 (PB1)
- new net: C13.1, R5.1, U1.29 (PB15)
- new net: R7.2, U1.14 (PA6)
- new net: C11.1, R3.1, U1.25 (PB11)
- new net: C12.1, R4.1, U1.27 (PB13)
- new net: J1.A5 (CC1), R1.1
- new net +3.3V: BOOT_SW1.2 (B), C1.2, C16.2, C17.2, C2.2, C3.2, C4.2, C5.2, J3.2 (Pin_2), R11.1, U1.1 (VBAT), U1.24 (VDD), U1.36 (VDD), U1.48 (VDD), U3.5 (OUT)
- new net +3.3VA: C18.2, C6.2, C7.2, C8.2, R11.2, U1.20 (VREF+), U1.21 (VDDA)
- new net +5V: C15.2, F1.2, J2.1 (Pin_1), J3.1 (Pin_1), U2.5 (VBUS), U3.1 (IN), U3.3 (EN)
- new net +5V_USB: F1.1, J1.A4 (VBUS), J1.A9 (VBUS), J1.B4 (VBUS), J1.B9 (VBUS)
- new net ADC0_IN: R3.2
- new net ADC1_IN: R4.2
- new net ADC2_IN: R5.2
- new net ADC3_IN: R6.2
- new net BOOT0: BOOT_SW1.1 (A), R12.1, U1.45 (PB8)
- new net D+: J2.3 (Pin_3), U1.34 (PA12), U2.1 (I/O1)
- new net D-: J2.2 (Pin_2), U1.33 (PA11), U2.3 (I/O2)
- new net DISCHARGE0: U1.26 (PB12)
- new net DISCHARGE1: U1.28 (PB14)
- new net DISCHARGE2: U1.30 (PA8)
- new net DISCHARGE3: U1.32 (PA10)
- new net DM_USB: J1.A7 (D-), J1.B7 (D-), U2.4 (I/O2)
- new net DP_USB: J1.A6 (D+), J1.B6 (D+), U2.6 (I/O1)
- new net GND: C1.1, C10.1, C11.2, C12.2, C13.2, C14.2, C15.1, C16.1, C17.1, C18.1, C19.1, C2.1, C3.1, C4.1, C5.1, C6.1, C7.1, C8.1, C9.1, J1.A1 (GND), J1.A12 (GND), J1.B1 (GND), J1.B12 (GND), J1.S1 (SHIELD), J2.4 (Pin_4), J3.4 (Pin_4), R1.2, R12.2, R2.2, RESET_SW1.2 (B), U1.19 (VSSA), U1.23 (VSS), U1.35 (VSS), U1.47 (VSS), U2.2 (GND), U3.2 (GND), Y1.2, Y1.4
- new net MUX0_EN: U1.43 (PB6)
- new net MUX1_EN: U1.44 (PB7)
- new net MUX_S0: U1.41 (PB4)
- new net MUX_S1: U1.42 (PB5)
- new net PWM: U1.9 (PA1)
- new net RESET: C19.2, J3.8 (Pin_8), RESET_SW1.1 (A), U1.7 (PG10)
- new net ROW0: R7.1
- new net ROW1: R8.1
- new net ROW2: R9.1
- new net ROW3: R10.1
- new net SWCLK: J3.6 (Pin_6), U1.38 (PA14)
- new net SWDIO: J3.7 (Pin_7), U1.37 (PA13)
- new net SWO: J3.5 (Pin_5), U1.40 (PB3)
- no-connect marks 0 -> 5
Other:
- added sheet Romashka EC MATRIX (Romashka EC MATRIX.kicad_sch)
- added sheet Romashka EC MUX & OPAMP (Romashka EC MUX & OPAMP.kicad_sch)
- note added: "5 - ADC1 6 - ADC2 8 - ADC12 9 - ADC12 10 - ADC1 11 - ADC1 12 - ADC2 13 - ADC2 14 - ADC2 15 - ADC2 16 - ADC3/ADC1 17 - ADC3/ADC1 18 - ADC2 25 - ADC12 26 - ADC4/ADC1 27 - ADC3 28 - ADC4/ADC1 29 - ADC4/ADC2 30 - ADC5 31 - ADC5"
