File: Romashka EC/Romashka EC MATRIX.kicad_sch (KiCad schematic)
At the start: 65 parts, among them SW1 EC_SW, SW10 EC_SW, SW11 EC_SW, SW12 EC_SW, SW13 EC_SW, SW14 EC_SW, SW15 EC_SW, SW16 EC_SW, SW17 EC_SW, SW18 EC_SW, SW19 EC_SW, SW2 EC_SW, SW20 EC_SW, SW21 EC_SW, SW22 EC_SW, SW23 EC_SW, SW24 EC_SW, SW25 EC_SW, SW26 EC_SW, SW27 EC_SW, SW28 EC_SW, SW29 EC_SW, SW3 EC_SW, SW30 EC_SW, SW31 EC_SW, SW32 EC_SW, SW33 EC_SW, SW34 EC_SW, SW35 EC_SW, SW36 EC_SW, SW37 EC_SW, SW38 EC_SW, SW39 EC_SW, SW4 EC_SW, SW40 EC_SW, SW41 EC_SW, SW42 EC_SW, SW43 EC_SW, SW44 EC_SW, SW45 EC_SW, SW46 EC_SW, SW47 EC_SW, SW48 EC_SW, SW49 EC_SW, SW5 EC_SW, SW6 EC_SW, SW7 EC_SW, SW8 EC_SW, SW9 EC_SW

Commit message: 20.04.2026: setup
Parts:
- SW1, SW10, SW13, SW14, SW15, SW16, SW17, SW18, SW19, SW2, SW20, SW21, SW22, SW24, SW25, SW26, SW28, SW29, SW3, SW30, SW31, SW32, SW4, SW42, SW5, SW8, SW9: footprint Kicad footprints:ecs_pad_1U_hybrid_hotswap_V2 -> Kicad footprints:ecs_pad_1U_hybrid_hotswap_V3
- SW11, SW12, SW23, SW35, SW38, SW40, SW6, SW7: footprint Kicad footprints:ecs_pad_1U_hybrid_hotswap_V2 -> Kicad footprints:ecs_pad_1U_hybrid_hotswap_V3_switched_sides
- SW27: footprint Kicad footprints:ecs_pad_1U_hybrid_hotswap_V2_switched_sides -> Kicad footprints:ecs_pad_1U_hybrid_hotswap_V3
- SW36, SW43, SW44, SW45, SW47: footprint Kicad footprints:ecs_pad_hybrid_hotswap_2.381_V2 -> Kicad footprints:ecs_pad_hybrid_hotswap_2.381_V3
- SW39: footprint Kicad footprints:ecs_pad_1U_hybrid_hotswap_V2_switched_sides -> Kicad footprints:ecs_pad_1U_hybrid_hotswap_V3_switched_sides
Changed lines of the file:
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@@
 			)
 		)
-		(property "Footprint" "Kicad footprints:ecs_pad_1U_hybrid_hotswap_V2"
+		(property "Footprint" "Kicad footprints:ecs_pad_1U_hybrid_hotswap_V3"
 			(at 58.42 60.96 0)
 			(effects
@@
 			)
 		)
-		(property "Footprint" "Kicad footprints:ecs_pad_1U_hybrid_hotswap_V2"
+		(property "Footprint" "Kicad footprints:ecs_pad_1U_hybrid_hotswap_V3"
 			(at 41.91 60.96 0)
 			(effects
@@
 			)
 		)
-		(property "Footprint" "Kicad footprints:ecs_pad_1U_hybrid_hotswap_V2"
+		(property "Footprint" "Kicad footprints:ecs_pad_1U_hybrid_hotswap_V3"
 			(at 173.99 45.72 0)
 			(effects
@@
 			)
 		)
-		(property "Footprint" "Kicad footprints:ecs_pad_hybrid_hotswap_2.381_V2"
+		(property "Footprint" "Kicad footprints:ecs_pad_hybrid_hotswap_2.381_V3"
 			(at 58.42 91.44 0)
 			(effects
@@
 			)
 		)
-		(property "Footprint" "Kicad footprints:ecs_pad_1U_hybrid_hotswap_V2"
+		(property "Footprint" "Kicad footprints:ecs_pad_1U_hybrid_hotswap_V3_switched_sides"
 			(at 157.48 91.44 0)
 			(effects
@@
 			)
 		)
-		(property "Footprint" "Kicad footprints:ecs_pad_1U_hybrid_hotswap_V2"
+		(property "Footprint" "Kicad footprints:ecs_pad_1U_hybrid_hotswap_V3"
 			(at 190.5 91.44 0)
 			(effects
@@
 					(size 1.27 1.27)
 				)
+				(hide yes)
 			)
 		)
@@
 					(size 1.27 1.27)
 				)
+				(hide yes)
 			)
 		)
@@
 			)
 		)
-		(property "Footprint" "Kicad footprints:ecs_pad_1U_hybrid_hotswap_V2"
+		(property "Footprint" "Kicad footprints:ecs_pad_1U_hybrid_hotswap_V3"
 			(at 74.93 76.2 0)
 			(effects
@@
 			)
 		)
-		(property "Footprint" "Kicad footprints:ecs_pad_1U_hybrid_hotswap_V2"
+		(property "Footprint" "Kicad footprints:ecs_pad_1U_hybrid_hotswap_V3_switched_sides"
 			(at 140.97 45.72 0)
 			(effects
@@
 					(size 1.27 1.27)
 				)
+				(hide yes)
 			)
 		)
@@
 					(size 1.27 1.27)
 				)
+				(hide yes)
 			)
 		)
@@
 			)
 		)
-		(property "Footprint" "Kicad footprints:ecs_pad_1U_hybrid_hotswap_V2"
+		(property "Footprint" "Kicad footprints:ecs_pad_1U_hybrid_hotswap_V3"
 			(at 74.93 45.72 0)
 			(effects
@@
 			)
 		)
-		(property "Footprint" "Kicad footprints:ecs_pad_hybrid_hotswap_2.381_V2"
+		(property "Footprint" "Kicad footprints:ecs_pad_hybrid_hotswap_2.381_V3"
 			(at 173.99 106.68 0)
 			(effects
@@
 			)
 		)
-		(property "Footprint" "Kicad footprints:ecs_pad_1U_hybrid_hotswap_V2"
+		(property "Footprint" "Kicad footprints:ecs_pad_1U_hybrid_hotswap_V3_switched_sides"
 			(at 207.01 60.96 0)
 			(effects
@@
 			)
 		)
-		(property "Footprint" "Kicad footprints:ecs_pad_1U_hybrid_hotswap_V2"
+		(property "Footprint" "Kicad footprints:ecs_pad_1U_hybrid_hotswap_V3"
 			(at 41.91 76.2 0)
 			(effects
@@
 			)
 		)
-		(property "Footprint" "Kicad footprints:ecs_pad_1U_hybrid_hotswap_V2"
+		(property "Footprint" "Kicad footprints:ecs_pad_1U_hybrid_hotswap_V3"
 			(at 107.95 60.96 0)
 			(effects
@@
 			)
 		)
-		(property "Footprint" "Kicad footprints:ecs_pad_1U_hybrid_hotswap_V2"
+		(property "Footprint" "Kicad footprints:ecs_pad_1U_hybrid_hotswap_V3"
 			(at 140.97 76.2 0)
 			(effects
@@
 			)
 		)
-		(property "Footprint" "Kicad footprints:ecs_pad_1U_hybrid_hotswap_V2"
+		(property "Footprint" "Kicad footprints:ecs_pad_1U_hybrid_hotswap_V3"
 			(at 173.99 60.96 0)
 			(effects
@@
 			)
 		)
-		(property "Footprint" "Kicad footprints:ecs_pad_1U_hybrid_hotswap_V2"
+		(property "Footprint" "Kicad footprints:ecs_pad_1U_hybrid_hotswap_V3"
 			(at 124.46 76.2 0)
 			(effects
@@
 			)
 		)
-		(property "Footprint" "Kicad footprints:ecs_pad_1U_hybrid_hotswap_V2"
+		(property "Footprint" "Kicad footprints:ecs_pad_1U_hybrid_hotswap_V3"
 			(at 41.91 45.72 0)
 			(effects
@@
 			)
 		)
-		(property "Footprint" "Kicad footprints:ecs_pad_1U_hybrid_hotswap_V2"
+		(property "Footprint" "Kicad footprints:ecs_pad_1U_hybrid_hotswap_V3"
 			(at 190.5 60.96 0)
 			(effects
@@
 			)
 		)
-		(property "Footprint" "Kicad footprints:ecs_pad_1U_hybrid_hotswap_V2"
+		(property "Footprint" "Kicad footprints:ecs_pad_1U_hybrid_hotswap_V3"
 			(at 157.48 76.2 0)
 			(effects
@@
 					(size 1.27 1.27)
 				)
+				(hide yes)
 			)
 		)
@@
 					(size 1.27 1.27)
 				)
+				(hide yes)
 			)
 		)
@@
 			)
 		)
-		(property "Footprint" "Kicad footprints:ecs_pad_1U_hybrid_hotswap_V2"
+		(property "Footprint" "Kicad footprints:ecs_pad_1U_hybrid_hotswap_V3_switched_sides"
 			(at 207.01 45.72 0)
 			(effects
@@
 			)
 		)
-		(property "Footprint" "Kicad footprints:ecs_pad_1U_hybrid_hotswap_V2_switched_sides"
+		(property "Footprint" "Kicad footprints:ecs_pad_1U_hybrid_hotswap_V3"
 			(at 91.44 76.2 0)
 			(effects
@@
 			)
 		)
-		(property "Footprint" "Kicad footprints:ecs_pad_1U_hybrid_hotswap_V2"
+		(property "Footprint" "Kicad footprints:ecs_pad_1U_hybrid_hotswap_V3"
 			(at 107.95 45.72 0)
 			(effects
@@
 			)
 		)
-		(property "Footprint" "Kicad footprints:ecs_pad_1U_hybrid_hotswap_V2"
+		(property "Footprint" "Kicad footprints:ecs_pad_1U_hybrid_hotswap_V3"
 			(at 91.44 45.72 0)
 			(effects
@@
 			)
 		)
-		(property "Footprint" "Kicad footprints:ecs_pad_hybrid_hotswap_2.381_V2"
+		(property "Footprint" "Kicad footprints:ecs_pad_hybrid_hotswap_2.381_V3"
 			(at 190.5 73.66 0)
 			(effects
@@
 			)
 		)
-		(property "Footprint" "Kicad footprints:ecs_pad_1U_hybrid_hotswap_V2"
+		(property "Footprint" "Kicad footprints:ecs_pad_1U_hybrid_hotswap_V3"
 			(at 58.42 76.2 0)
 			(effects
@@
 			)
 		)
-		(property "Footprint" "Kicad footprints:ecs_pad_1U_hybrid_hotswap_V2"
+		(property "Footprint" "Kicad footprints:ecs_pad_1U_hybrid_hotswap_V3_switched_sides"
 			(at 91.44 91.44 0)
 			(effects
@@
 			)
 		)
-		(property "Footprint" "Kicad footprints:ecs_pad_1U_hybrid_hotswap_V2"
+		(property "Footprint" "Kicad footprints:ecs_pad_1U_hybrid_hotswap_V3"
 			(at 58.42 45.72 0)
 			(effects
@@
 			)
 		)
-		(property "Footprint" "Kicad footprints:ecs_pad_hybrid_hotswap_2.381_V2"
+		(property "Footprint" "Kicad footprints:ecs_pad_hybrid_hotswap_2.381_V3"
 			(at 74.93 106.68 0)
 			(effects
@@
 			)
 		)
-		(property "Footprint" "Kicad footprints:ecs_pad_1U_hybrid_hotswap_V2"
+		(property "Footprint" "Kicad footprints:ecs_pad_1U_hybrid_hotswap_V3"
 			(at 157.48 45.72 0)
 			(effects
@@
 			)
 		)
-		(property "Footprint" "Kicad footprints:ecs_pad_1U_hybrid_hotswap_V2"
+		(property "Footprint" "Kicad footprints:ecs_pad_1U_hybrid_hotswap_V3"
 			(at 157.48 60.96 0)
 			(effects
@@
 			)
 		)
-		(property "Footprint" "Kicad footprints:ecs_pad_1U_hybrid_hotswap_V2"
+		(property "Footprint" "Kicad footprints:ecs_pad_1U_hybrid_hotswap_V3"
 			(at 91.44 60.96 0)
 			(effects
@@
 			)
 		)
-		(property "Footprint" "Kicad footprints:ecs_pad_1U_hybrid_hotswap_V2"
+		(property "Footprint" "Kicad footprints:ecs_pad_1U_hybrid_hotswap_V3"
 			(at 107.95 76.2 0)
 			(effects
@@
 			)
 		)
-		(property "Footprint" "Kicad footprints:ecs_pad_1U_hybrid_hotswap_V2"
+		(property "Footprint" "Kicad footprints:ecs_pad_1U_hybrid_hotswap_V3"
 			(at 74.93 60.96 0)
 			(effects
@@
 			)
 		)
-		(property "Footprint" "Kicad footprints:ecs_pad_1U_hybrid_hotswap_V2"
+		(property "Footprint" "Kicad footprints:ecs_pad_1U_hybrid_hotswap_V3"
 			(at 190.5 45.72 0)
 			(effects
@@
 			)
 		)
-		(property "Footprint" "Kicad footprints:ecs_pad_1U_hybrid_hotswap_V2"
+		(property "Footprint" "Kicad footprints:ecs_pad_1U_hybrid_hotswap_V3"
 			(at 173.99 76.2 0)
 			(effects
@@
 					(size 1.27 1.27)
 				)
+				(hide yes)
 			)
 		)
@@
 					(size 1.27 1.27)
 				)
+				(hide yes)
 			)
 		)
@@
 			)
 		)
-		(property "Footprint" "Kicad footprints:ecs_pad_1U_hybrid_hotswap_V2"
+		(property "Footprint" "Kicad footprints:ecs_pad_1U_hybrid_hotswap_V3"
 			(at 124.46 60.96 0)
 			(effects
@@
 			)
 		)
-		(property "Footprint" "Kicad footprints:ecs_pad_1U_hybrid_hotswap_V2"
+		(property "Footprint" "Kicad footprints:ecs_pad_1U_hybrid_hotswap_V3"
 			(at 140.97 60.96 0)
 			(effects
@@
 			)
 		)
-		(property "Footprint" "Kicad footprints:ecs_pad_1U_hybrid_hotswap_V2"
+		(property "Footprint" "Kicad footprints:ecs_pad_1U_hybrid_hotswap_V3_switched_sides"
 			(at 207.01 76.2 0)
 			(effects
@@
 			)
 		)
-		(property "Footprint" "Kicad footprints:ecs_pad_hybrid_hotswap_2.381_V2"
+		(property "Footprint" "Kicad footprints:ecs_pad_hybrid_hotswap_2.381_V3"
 			(at 207.01 88.9 0)
 			(effects
@@
 			)
 		)
-		(property "Footprint" "Kicad footprints:ecs_pad_1U_hybrid_hotswap_V2"
+		(property "Footprint" "Kicad footprints:ecs_pad_1U_hybrid_hotswap_V3_switched_sides"
 			(at 41.91 91.44 0)
 			(effects
@@
 			)
 		)
-		(property "Footprint" "Kicad footprints:ecs_pad_1U_hybrid_hotswap_V2_switched_sides"
+		(property "Footprint" "Kicad footprints:ecs_pad_1U_hybrid_hotswap_V3_switched_sides"
 			(at 140.97 91.44 0)
 			(effects
@@
 					(size 1.27 1.27)
 				)
+				(hide yes)
 			)
 		)
@@
 					(size 1.27 1.27)
 				)
+				(hide yes)
 			)
 		)
@@
 			)
 		)
-		(property "Footprint" "Kicad footprints:ecs_pad_1U_hybrid_hotswap_V2"
+		(property "Footprint" "Kicad footprints:ecs_pad_1U_hybrid_hotswap_V3_switched_sides"
 			(at 124.46 45.72 0)
 			(effects
@@
 					(size 1.27 1.27)
 				)
+				(hide yes)
 			)
 		)
@@
 					(size 1.27 1.27)
 				)
+				(hide yes)
 			)
 		)

Commit message: 21.04.2026: footprints
Parts:
- SW23: footprint Kicad footprints:ecs_pad_1U_hybrid_hotswap_V3_switched_sides -> Kicad footprints:ecs_pad_1U_hybrid_hotswap_V3
- SW49: footprint Kicad footprints:ecs_pad_1U_hybrid_hotswap_7.144 -> Kicad footprints:ecs_pad_hybrid_hotswap_7.144_V3
Changed lines of the file:
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@@
 			)
 		)
-		(property "Footprint" "Kicad footprints:ecs_pad_1U_hybrid_hotswap_7.144"
+		(property "Footprint" "Kicad footprints:ecs_pad_hybrid_hotswap_7.144_V3"
 			(at 124.46 105.41 0)
 			(effects
@@
 			)
 		)
-		(property "Footprint" "Kicad footprints:ecs_pad_1U_hybrid_hotswap_V3_switched_sides"
+		(property "Footprint" "Kicad footprints:ecs_pad_1U_hybrid_hotswap_V3"
 			(at 207.01 76.2 0)
 			(effects
