File: Romashka EC non-matrix/OPAMP.kicad_sch (KiCad schematic)
At the start: 30 parts, among them U10 OPA2365, U11 OPA2365, U12 OPA2365

Commit message: 21.04.2026 09:06
Parts:
- removed C26, C30, C33: 100nF, Capacitor_SMD:C_0402_1005Metric, symbol Device:C_Small
- removed C27, C28, C29, C31, C32, C34: 50-100pF, Capacitor_SMD:C_0402_1005Metric, symbol Device:C_Small
- removed R13, R17, R20, R23, R26, R29: 33K, Resistor_SMD:R_0603_1608Metric, symbol Device:R_Small
- removed R14, R15, R16, R18, R19, R21, R22, R24, R25, R27, R28, R30: 330R, Resistor_SMD:R_0603_1608Metric, symbol Device:R_Small
- removed U10, U11, U12: OPA2365, Package_SO:SOIC-8_3.9x4.9mm_P1.27mm, symbol Amplifier_Operational:OPA2376xxD
