File: Romashka EC non-matrix/Romashka EC non-matrix.kicad_sch (KiCad schematic)
At the start: 35 parts, among them J1 Daisy40, J2 JSB USB, J3 SOICbite, J4 JJ40, J5 RS40, U1 STM32G474CBTx, U2 USBLC6-2P6, U3 TPS7A2033, Y1 8Mhz 12pF

Commit message: 21.04.2026 09:06
Other:
- removed sheet OPAMP
Changed lines of the file:
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@@
-	)
-	(sheet
-		(at 228.6 73.025)
-		(size 36.83 36.195)
-		(exclude_from_sim no)
-		(in_bom yes)
-		(on_board yes)
-		(dnp no)
-		(fields_autoplaced yes)
-		(stroke
-			(width 0.1524)
-			(type solid)
-		)
-		(fill
-			(color 0 0 0 0.0000)
-		)
-		(property "Sheetname" "OPAMP"
-			(at 228.6 72.3134 0)
-			(effects
-				(font
-					(size 1.27 1.27)
-				)
-				(justify left bottom)
-			)
-		)
-		(property "Sheetfile" "OPAMP.kicad_sch"
-			(at 228.6 109.8046 0)
-			(effects
-				(font
-					(size 1.27 1.27)
-				)
-				(justify left top)
-			)
-		)
-		(instances
-			(project "Romashka EC non-matrix"
-				(path "/69f48e55-4bf1-48a7-a2c4-b2689bdf9720"
-					(page "3")
-				)
-			)
-		)
 	)
 	(sheet

Commit message: 22.04.2026
Parts:
- renumbered C17 to C15, C18 to C16, C19 to C17, C15 to C18, C16 to C19, J5 to J2, J4 to J3, J2 to J4, J3 to J5, R5 to R2, R2 to R3, R6 to R4, R3 to R5, R4 to R6
Connections:
- net DISCHARGE0 renamed COM5
- net DISCHARGE1 renamed COM4
- net DISCHARGE2 renamed COM3
- net DISCHARGE3 renamed COM2
- net DISCHARGE4 renamed COM1
- net DISCHARGE5 renamed COM0
Changed lines of the file:
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@@
 		)
 	)
-	(global_label "DISCHARGE4"
+	(global_label "COM4"
 		(shape input)
-		(at 170.18 95.25 180)
+		(at 170.18 102.87 180)
 		(fields_autoplaced yes)
 		(effects
@@
 		)
 		(property "Intersheetrefs" "${INTERSHEET_REFS}"
-			(at 155.5229 95.25 0)
+			(at 161.9334 102.87 0)
 			(effects
 				(font
@@
 		)
 	)
-	(global_label "DISCHARGE3"
+	(global_label "SWO"
 		(shape input)
-		(at 170.18 97.79 180)
+		(at 170.18 74.93 180)
 		(fields_autoplaced yes)
 		(effects
@@
 		)
 		(property "Intersheetrefs" "${INTERSHEET_REFS}"
-			(at 155.5229 97.79 0)
+			(at 163.2034 74.93 0)
 			(effects
 				(font
@@
 		)
 	)
-	(global_label "DISCHARGE1"
+	(global_label "DRIVE_MUX5"
 		(shape input)
-		(at 170.18 102.87 180)
+		(at 205.74 52.07 0)
 		(fields_autoplaced yes)
 		(effects
@@
 				(size 1.27 1.27)
 			)
-			(justify right)
+			(justify left)
 		)
 		(property "Intersheetrefs" "${INTERSHEET_REFS}"
-			(at 155.5229 102.87 0)
+			(at 220.2761 52.07 0)
 			(effects
 				(font
 					(size 1.27 1.27)
 				)
-				(justify right)
+				(justify left)
 				(hide yes)
 			)
 		)
 	)
-	(global_label "SWO"
+	(global_label "DRIVE_MUX4"
 		(shape input)
-		(at 170.18 74.93 180)
+		(at 205.74 49.53 0)
 		(fields_autoplaced yes)
 		(effects
@@
 				(size 1.27 1.27)
 			)
-			(justify right)
+			(justify left)
 		)
 		(property "Intersheetrefs" "${INTERSHEET_REFS}"
-			(at 163.2034 74.93 0)
+			(at 220.2761 49.53 0)
 			(effects
 				(font
 					(size 1.27 1.27)
 				)
-				(justify right)
+				(justify left)
 				(hide yes)
 			)
 		)
 	)
-	(global_label "DRIVE_MUX5"
+	(global_label "MUX_S2"
 		(shape input)
-		(at 205.74 52.07 0)
+		(at 170.18 67.31 180)
 		(fields_autoplaced yes)
 		(effects
@@
 				(size 1.27 1.27)
 			)
-			(justify left)
+			(justify right)
 		)
 		(property "Intersheetrefs" "${INTERSHEET_REFS}"
-			(at 220.2761 52.07 0)
+			(at 159.8168 67.31 0)
 			(effects
 				(font
 					(size 1.27 1.27)
 				)
-				(justify left)
+				(justify right)
 				(hide yes)
 			)
 		)
 	)
-	(global_label "DRIVE_MUX4"
+	(global_label "COM0"
 		(shape input)
-		(at 205.74 49.53 0)
+		(at 170.18 92.71 180)
 		(fields_autoplaced yes)
 		(effects
@@
 				(size 1.27 1.27)
 			)
-			(justify left)
+			(justify right)
 		)
 		(property "Intersheetrefs" "${INTERSHEET_REFS}"
-			(at 220.2761 49.53 0)
+			(at 161.9334 92.71 0)
 			(effects
 				(font
 					(size 1.27 1.27)
 				)
-				(justify left)
+				(justify right)
 				(hide yes)
 			)
 		)
 	)
-	(global_label "MUX_S2"
+	(global_label "COM3"
 		(shape input)
-		(at 170.18 67.31 180)
+		(at 170.18 100.33 180)
 		(fields_autoplaced yes)
 		(effects
@@
 		)
 		(property "Intersheetrefs" "${INTERSHEET_REFS}"
-			(at 159.8168 67.31 0)
+			(at 161.9334 100.33 0)
 			(effects
 				(font
@@
 		)
 	)
-	(global_label "DISCHARGE2"
-		(shape input)
-		(at 170.18 100.33 180)
-		(fields_autoplaced yes)
-		(effects
-			(font
-				(size 1.27 1.27)
-			)
-			(justify right)
-		)
-		(property "Intersheetrefs" "${INTERSHEET_REFS}"
-			(at 155.5229 100.33 0)
-			(effects
-				(font
-					(size 1.27 1.27)
-				)
-				(justify right)
-				(hide yes)
-			)
-		)
-	)
 	(global_label "SWDIO"
 		(shape input)
@@
 		)
 	)
-	(global_label "DISCHARGE5"
+	(global_label "RESET"
 		(shape input)
-		(at 170.18 92.71 180)
+		(at 153.67 175.26 180)
 		(fields_autoplaced yes)
 		(effects
@@
 		)
 		(property "Intersheetrefs" "${INTERSHEET_REFS}"
-			(at 155.5229 92.71 0)
+			(at 144.9397 175.26 0)
 			(effects
 				(font
@@
 		)
 	)
-	(global_label "DISCHARGE0"
+	(global_label "COM5"
 		(shape input)
 		(at 170.18 105.41 180)
@@
 		)
 		(property "Intersheetrefs" "${INTERSHEET_REFS}"
-			(at 155.5229 105.41 0)
-			(effects
-				(font
-					(size 1.27 1.27)
-				)
-				(justify right)
-				(hide yes)
-			)
-		)
-	)
-	(global_label "RESET"
-		(shape input)
-		(at 153.67 175.26 180)
-		(fields_autoplaced yes)
-		(effects
-			(font
-				(size 1.27 1.27)
-			)
-			(justify right)
-		)
-		(property "Intersheetrefs" "${INTERSHEET_REFS}"
-			(at 144.9397 175.26 0)
+			(at 161.9334 105.41 0)
 			(effects
 				(font
@@
 		)
 	)
+	(global_label "COM2"
+		(shape input)
+		(at 170.18 97.79 180)
+		(fields_autoplaced yes)
+		(effects
+			(font
+				(size 1.27 1.27)
+			)
+			(justify right)
+		)
+		(property "Intersheetrefs" "${INTERSHEET_REFS}"
+			(at 161.9334 97.79 0)
+			(effects
+				(font
+					(size 1.27 1.27)
+				)
+				(justify right)
+				(hide yes)
+			)
+		)
+	)
+	(global_label "COM1"
+		(shape input)
+		(at 170.18 95.25 180)
+		(fields_autoplaced yes)
+		(effects
+			(font
+				(size 1.27 1.27)
+			)
+			(justify right)
+		)
+		(property "Intersheetrefs" "${INTERSHEET_REFS}"
+			(at 161.9334 95.25 0)
+			(effects
+				(font
+					(size 1.27 1.27)
+				)
+				(justify right)
+				(hide yes)
+			)
+		)
+	)
 	(global_label "ADC5"
 		(shape input)
@@
 		(on_board yes)
 		(dnp no)
-		(property "Reference" "R2"
+		(property "Reference" "R3"
 			(at 55.88 39.37 90)
 			(effects
@@
 			(project "Romashka EC non-matrix"
 				(path "/69f48e55-4bf1-48a7-a2c4-b2689bdf9720"
-					(reference "R2")
+					(reference "R3")
 					(unit 1)
 				)
@@
 		(on_board yes)
 		(dnp no)
-		(property "Reference" "R4"
+		(property "Reference" "R6"
 			(at 55.88 93.98 90)
 			(effects
@@
 			(project "Romashka EC non-matrix"
 				(path "/69f48e55-4bf1-48a7-a2c4-b2689bdf9720"
-					(reference "R4")
+					(reference "R6")
 					(unit 1)
 				)
@@
 		(dnp no)
 		(fields_autoplaced yes)
-		(property "Reference" "R5"
+		(property "Reference" "R2"
 			(at 104.14 26.67 90)
 			(effects
@@
 			(project "Romashka EC non-matrix"
 				(path "/69f48e55-4bf1-48a7-a2c4-b2689bdf9720"
-					(reference "R5")
+					(reference "R2")
 					(unit 1)
 				)
@@
 		(dnp no)
 		(fields_autoplaced yes)
-		(property "Reference" "J3"
+		(property "Reference" "J5"
 			(at 196.85 147.3199 0)
 			(effects
@@
 			(project "Romashka EC non-matrix"
 				(path "/69f48e55-4bf1-48a7-a2c4-b2689bdf9720"
-					(reference "J3")
+					(reference "J5")
 					(unit 1)
 				)
@@
 		(on_board yes)
 		(dnp no)
-		(property "Reference" "R6"
+		(property "Reference" "R4"
 			(at 109.22 39.37 90)
 			(effects
@@
 			(project "Romashka EC non-matrix"
 				(path "/69f48e55-4bf1-48a7-a2c4-b2689bdf9720"
-					(reference "R6")
+					(reference "R4")
 					(unit 1)
 				)
@@
 		(on_board yes)
 		(dnp no)
-		(property "Reference" "C19"
+		(property "Reference" "C17"
 			(at 152.4 177.7935 0)
 			(effects
@@
 			(project "Romashka EC non-matrix"
 				(path "/69f48e55-4bf1-48a7-a2c4-b2689bdf9720"
-					(reference "C19")
+					(reference "C17")
 					(unit 1)
 				)
@@
 		(dnp no)
 		(fields_autoplaced yes)
-		(property "Reference" "J5"
+		(property "Reference" "J2"
 			(at 85.09 19.05 0)
 			(effects
@@
 			(project "Romashka EC non-matrix"
 				(path "/69f48e55-4bf1-48a7-a2c4-b2689bdf9720"
-					(reference "J5")
+					(reference "J2")
 					(unit 1)
 				)
@@
 		(on_board yes)
 		(dnp no)
-		(property "Reference" "C16"
+		(property "Reference" "C19"
 			(at 49.53 182.8735 0)
 			(effects
@@
 			(project "Romashka EC non-matrix"
 				(path "/69f48e55-4bf1-48a7-a2c4-b2689bdf9720"
-					(reference "C16")
+					(reference "C19")
 					(unit 1)
 				)
@@
 		(dnp no)
 		(fields_autoplaced yes)
-		(property "Reference" "C15"
+		(property "Reference" "C18"
 			(at 29.21 182.8735 0)
 			(effects
@@
 			(project "Romashka EC non-matrix"
 				(path "/69f48e55-4bf1-48a7-a2c4-b2689bdf9720"
-					(reference "C15")
+					(reference "C18")
 					(unit 1)
 				)
@@
 		(dnp no)
 		(fields_autoplaced yes)
-		(property "Reference" "J4"
+		(property "Reference" "J3"
 			(at 31.75 73.66 0)
 			(effects
@@
 			(project "Romashka EC non-matrix"
 				(path "/69f48e55-4bf1-48a7-a2c4-b2689bdf9720"
-					(reference "J4")
+					(reference "J3")
 					(unit 1)
 				)
@@
 		(dnp no)
 		(fields_autoplaced yes)
-		(property "Reference" "J2"
+		(property "Reference" "J4"
 			(at 256.54 146.0499 0)
 			(effects
@@
 			(project "Romashka EC non-matrix"
 				(path "/69f48e55-4bf1-48a7-a2c4-b2689bdf9720"
-					(reference "J2")
+					(reference "J4")
 					(unit 1)
 				)
@@
 		(dnp no)
 		(fields_autoplaced yes)
-		(property "Reference" "R3"
+		(property "Reference" "R5"
 			(at 50.8 81.28 90)
 			(effects
@@
 			(project "Romashka EC non-matrix"
 				(path "/69f48e55-4bf1-48a7-a2c4-b2689bdf9720"
-					(reference "R3")
+					(reference "R5")
 					(unit 1)
 				)
@@
 		(on_board yes)
 		(dnp no)
-		(property "Reference" "C17"
+		(property "Reference" "C15"
 			(at 76.2 177.7935 0)
 			(effects
@@
 			(project "Romashka EC non-matrix"
 				(path "/69f48e55-4bf1-48a7-a2c4-b2689bdf9720"
-					(reference "C17")
+					(reference "C15")
 					(unit 1)
 				)
@@
 		(on_board yes)
 		(dnp no)
-		(property "Reference" "C18"
+		(property "Reference" "C16"
 			(at 93.98 177.7935 0)
 			(effects
@@
 			(project "Romashka EC non-matrix"
 				(path "/69f48e55-4bf1-48a7-a2c4-b2689bdf9720"
-					(reference "C18")
+					(reference "C16")
 					(unit 1)
 				)

Commit message: 22.04.2026 something something
Parts:
- removed C10, C9: 15pF, Capacitor_SMD:C_0402_1005Metric, symbol Device:C_Small
- removed Y1: 8Mhz 12pF, Crystal:Crystal_SMD_3225-4Pin_3.2x2.5mm, symbol Device:Crystal_GND24_Small
- added R27, R28, R29, R30, R31, R32, R33, R34, R35, R36, R37, R38: 330, Resistor_SMD:R_0603_1608Metric, symbol Device:R_Small
Connections:
- net ADC0: now also R27.2; no longer U1.46 (PB9)
- net ADC1: now also R28.2; no longer U1.14 (PA6)
- net ADC2: now also R29.2; no longer U1.15 (PA7)
- net ADC3: now also R30.2; no longer U1.30 (PA8)
- net ADC4: now also R31.2; no longer U1.31 (PA9)
- net ADC5: now also R32.2; no longer U1.32 (PA10)
- net MUX_S0: now also U1.43 (PB6); no longer U1.18 (PB2)
- net MUX_S1: now also U1.42 (PB5); no longer U1.17 (PB1)
- net MUX_S2: now also U1.41 (PB4); no longer U1.16 (PB0)
- net COM0: no longer names the net of U1.22 (PB10)
- net COM1: no longer names the net of U1.25 (PB11)
- net COM2: no longer names the net of U1.26 (PB12)
- net COM3: no longer names the net of U1.27 (PB13)
- net COM4: no longer names the net of U1.28 (PB14)
- net COM5: no longer names the net of U1.29 (PB15)
- net DRIVE_MUX0: no longer names the net of U1.8 (PA0)
- net DRIVE_MUX1: no longer names the net of U1.9 (PA1)
- net DRIVE_MUX2: no longer names the net of U1.10 (PA2)
- net DRIVE_MUX3: no longer names the net of U1.11 (PA3)
- net DRIVE_MUX4: no longer names the net of U1.12 (PA4)
- net DRIVE_MUX5: no longer names the net of U1.13 (PA5)
- new net MUX0_IN: R33.1
- new net MUX1_IN: R34.1
- new net MUX2_IN: R35.1
- new net MUX3_IN: R36.1
- new net MUX4_IN: R37.1
- new net MUX5_IN: R38.1
- no-connect marks 9 -> 11
Other:
- removed sheet MUX & MATRIX
- added sheet Logic (Logic.kicad_sch)
- moved on the sheet: C1, C2, C3, C4, C5, C6, C7, C8, J4, J5, U1

Commit message: 24.04.2026
Parts:
- removed R31, R32, R37, R38: 330, Resistor_SMD:R_0603_1608Metric, symbol Device:R_Small
- J2, J3, R2, R4: now not fitted; now left out of the parts list
- R19: renamed from R5; now not fitted; now left out of the parts list
- R20: renamed from R6; now not fitted; now left out of the parts list
- renumbered C15 to C13, C16 to C14, C17 to C15, C18 to C16, C19 to C17, J5 to J4, J4 to J5, R29 to R11, R30 to R12, R33 to R25, R34 to R26, R35 to R27, R36 to R28, R11 to R31, R12 to R32, R27 to R5, R28 to R6
Connections:
- net MUX_S0: now also U1.44 (PB7); no longer U1.43 (PB6)
- net MUX_S1: now also U1.43 (PB6); no longer U1.42 (PB5)
- net MUX_S2: now also U1.42 (PB5); no longer U1.41 (PB4)
- net at R28.2: now also U1.29 (PB15)
- net at R11.1: now also U1.10 (PA2)
- net at R12.1: now also U1.11 (PA3)
- net at R6.1: now also U1.9 (PA1)
- net at R25.2: now also U1.26 (PB12)
- net at R26.2: now also U1.27 (PB13)
- net DISCHARGE3: now reaches U1.12 (PA4)
- net DISCHARGE2: now reaches U1.13 (PA5)
- net DISCHARGE1: now reaches U1.14 (PA6)
- net DISCHARGE0: now reaches U1.15 (PA7)
- net at U1.28 (PB14): now also R27.2
- net at U1.8 (PA0): now also R5.1
- new net MUX_S3: U1.41 (PB4)
Other:
- moved on the sheet: R11, R12, R25, R26, R27, R28, R5, R6

Commit message: 28.04.2026
Connections:
- net ADC0: now also U1.15 (PA7)
- net ADC1: now also U1.26 (PB12)
- net ADC2: now also U1.28 (PB14)
- net ADC3: now also U1.9 (PA1)
- net DISCHARGE0: now also U1.13 (PA5); no longer U1.15 (PA7)
- net DISCHARGE1: now also U1.25 (PB11); no longer U1.14 (PA6)
- net DISCHARGE2: now also U1.27 (PB13); no longer U1.13 (PA5)
- net DISCHARGE3: now also U1.8 (PA0); no longer U1.12 (PA4)
- net at R28.2: no longer U1.29 (PB15)
- net at R11.1: no longer U1.10 (PA2)
- net at R12.1: no longer U1.11 (PA3)
- net at R6.1: no longer U1.9 (PA1)
- net at R25.2: no longer U1.26 (PB12)
- net at R26.2: no longer U1.27 (PB13)
- net at R27.2: no longer U1.28 (PB14)
- net at R5.1: no longer U1.8 (PA0)
Other:
- moved on the sheet: R11, R12, R25, R26, R27, R28, R5, R6

Commit message: 29.04.2026
Connections:
- net +3.3V: now also J4.8 (Pin_8); no longer J4.2 (Pin_2)
- net +5V: no longer J4.1 (Pin_1)
- net GND: now also J4.5 (Pin_5); no longer J4.4 (Pin_4)
- net RESET: now also J4.1 (Pin_1); no longer J4.8 (Pin_8)
- net SWCLK: now also J4.3 (Pin_3); no longer J4.6 (Pin_6)
- net SWDIO: now also J4.2 (Pin_2); no longer J4.7 (Pin_7)
- net SWO: now also J4.4 (Pin_4); no longer J4.5 (Pin_5)
- no-connect marks 11 -> 12
Changed lines of the file:
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@@
 	)
 	(no_connect
+		(at 212.09 93.98)
+	)
+	(no_connect
 		(at 212.09 58.42)
 	)
@@
 	(wire
 		(pts
-			(xy 195.58 135.89) (xy 200.66 135.89)
-		)
-		(stroke
-			(width 0)
-			(type default)
-		)
-	)
-	(wire
-		(pts
 			(xy 77.47 64.77) (xy 85.09 64.77)
 		)
@@
 	(wire
 		(pts
-			(xy 190.5 138.43) (xy 200.66 138.43)
+			(xy 189.23 135.89) (xy 200.66 135.89)
 		)
 		(stroke
@@
 		(lib_id "power:GND")
 		(at 189.23 143.51 0)
+		(mirror y)
 		(unit 1)
 		(exclude_from_sim no)
@@
 	(symbol
 		(lib_id "power:+3.3V")
-		(at 190.5 138.43 0)
+		(at 189.23 135.89 0)
 		(unit 1)
 		(exclude_from_sim no)
@@
 		(fields_autoplaced yes)
 		(property "Reference" "#PWR065"
-			(at 190.5 142.24 0)
+			(at 189.23 139.7 0)
 			(effects
 				(font
@@
 		)
 		(property "Value" "+3.3V"
-			(at 190.5 133.35 0)
+			(at 189.23 130.81 0)
 			(effects
 				(font
@@
 		)
 		(property "Footprint" ""
-			(at 190.5 138.43 0)
+			(at 189.23 135.89 0)
 			(effects
 				(font
@@
 		)
 		(property "Datasheet" ""
-			(at 190.5 138.43 0)
+			(at 189.23 135.89 0)
 			(effects
 				(font
@@
 		)
 		(property "Description" "Power symbol creates a global label with name \"+3.3V\""
-			(at 190.5 138.43 0)
+			(at 189.23 135.89 0)
 			(effects
 				(font
@@
 	(symbol
 		(lib_id "Connector_Generic:Conn_01x08")
-		(at 205.74 143.51 0)
+		(at 205.74 146.05 0)
+		(mirror x)
 		(unit 1)
 		(exclude_from_sim no)
@@
 		(fields_autoplaced yes)
 		(property "Reference" "J4"
-			(at 208.28 143.5099 0)
+			(at 208.28 146.0501 0)
 			(effects
 				(font
@@
 		)
 		(property "Value" "SOICbite"
-			(at 208.28 146.0499 0)
+			(at 208.28 143.5101 0)
 			(effects
 				(font
@@
 		)
 		(property "Footprint" "Kicad footprints:SOICbite_footprint"
-			(at 205.74 143.51 0)
+			(at 205.74 146.05 0)
 			(effects
 				(font
@@
 		)
 		(property "Datasheet" "~"
-			(at 205.74 143.51 0)
+			(at 205.74 146.05 0)
 			(effects
 				(font
@@
 		)
 		(property "Description" "Generic connector, single row, 01x08, script generated (kicad-library-utils/schlib/autogen/connector/)"
-			(at 205.74 143.51 0)
+			(at 205.74 146.05 0)
 			(effects
 				(font
@@
 					(unit 1)
 				)
-			)
-		)
-	)
-	(symbol
-		(lib_id "power:+5V")
-		(at 195.58 135.89 0)
-		(unit 1)
-		(exclude_from_sim no)
-		(in_bom yes)
-		(on_board yes)
-		(dnp no)
-		(fields_autoplaced yes)
-		(property "Reference" "#PWR014"
-			(at 195.58 139.7 0)
-			(effects
-				(font
-					(size 1.27 1.27)
-				)
-				(hide yes)
-			)
-		)
-		(property "Value" "+5V"
-			(at 195.58 130.81 0)
-			(effects
-				(font
-					(size 1.27 1.27)
-				)
-			)
-		)
-		(property "Footprint" ""
-			(at 195.58 135.89 0)
-			(effects
-				(font
-					(size 1.27 1.27)
-				)
-				(hide yes)
-			)
-		)
-		(property "Datasheet" ""
-			(at 195.58 135.89 0)
-			(effects
-				(font
-					(size 1.27 1.27)
-				)
-				(hide yes)
-			)
-		)
-		(property "Description" "Power symbol creates a global label with name \"+5V\""
-			(at 195.58 135.89 0)
-			(effects
-				(font
-					(size 1.27 1.27)
-				)
-				(hide yes)
-			)
-		)
-		(pin "1"
-		)
-		(instances
-			(project "Romashka EC non-matrix"
-				(path "/69f48e55-4bf1-48a7-a2c4-b2689bdf9720"
-					(reference "#PWR014")
-					(unit 1)
-				)

Commit message: 30.04.2026
Parts:
- removed C13: 1uF, Capacitor_SMD:C_0603_1608Metric, symbol Device:C_Small
- removed R11, R12, R25, R26, R27, R28, R5, R6: 330, Resistor_SMD:R_0603_1608Metric, symbol Device:R_Small
- renumbered C14 to C13, C15 to C14, C16 to C15, C17 to C16, J5 to J4, J4 to J5, R31 to R11, R32 to R12, R19 to R5, R20 to R6
Connections:
- net BOOT0: now also J5.1 (Pin_1)
- net MUX0_IN: now also U1.11 (PA3)
- net MUX1_IN: now also U1.10 (PA2)
- net MUX2_IN: now also U1.32 (PA10)
- net MUX3_IN: now also U1.31 (PA9)
- net RESET: now also J5.6 (Pin_6); no longer J5.1 (Pin_1)
- net SWDIO: now also J5.4 (Pin_4); no longer J5.2 (Pin_2)
- net SWO: now also J5.2 (Pin_2); no longer J5.4 (Pin_4)
