File: Romashka EC non-matrix/Romashka EC non-matrix.kicad_sch (KiCad schematic)
At the start: 31 parts, among them J1 Daisy40, J2 RS40, J3 JJ40, J4 JSB USB, J5 SOICbite, U1 STM32G474CBTx, U2 USBLC6-2P6, U3 TPS7A2033

Commit message: 14.05.2026
Parts:
- added C17, C26: 15pF, Capacitor_SMD:C_0402_1005Metric, symbol Device:C_Small
- added Y1: Crystal_GND24_Small, Crystal:Crystal_SMD_3225-4Pin_3.2x2.5mm, symbol Device:Crystal_GND24_Small
Connections:
- net +3.3V: now also J5.7 (Pin_7); no longer J5.8 (Pin_8)
- net GND: now also C17.1, C26.1, Y1.2, Y1.4
- net RESET: now also J5.8 (Pin_8); no longer J5.6 (Pin_6)
- net at U1.5 (PF0): now also C17.2, Y1.3
- net at U1.6 (PF1): now also C26.2, Y1.1
- no-connect marks 12 -> 10

Commit message: 17.05.2026
Parts:
- added H1, H2, H3, H4, H5, H6: MountingHole, Kicad footprints:m2 hole, symbol Mechanical:MountingHole
Connections:
- net ADC0: now also U1.14 (PA6); no longer U1.15 (PA7)
- net ADC1: now also U1.27 (PB13); no longer U1.26 (PB12)
- net ADC2: now also U1.12 (PA4); no longer U1.28 (PB14)
- net ADC3: now also U1.28 (PB14); no longer U1.9 (PA1)
- net DISCHARGE1: now also U1.46 (PB9); no longer U1.25 (PB11)
- net DISCHARGE2: now also U1.9 (PA1); no longer U1.27 (PB13)
- net DISCHARGE3: now also U1.26 (PB12); no longer U1.8 (PA0)

Commit message: 18.05.2026
Connections:
- net DM_USB renamed USB_D-
- net DP_USB renamed USB_D+

Commit message: 19.05.2026
Connections:
- net +3.3V: now also J5.6 (Pin_6); no longer J5.7 (Pin_7)
- net GND: now also J5.7 (Pin_7)
Changed lines of the file:
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@@
+	)
+	(junction
+		(at 189.23 143.51)
+		(diameter 0)
+		(color 0 0 0 0)
 	)
 	(junction
@@
 	(wire
 		(pts
+			(xy 189.23 138.43) (xy 189.23 143.51)
+		)
+		(stroke
+			(width 0)
+			(type default)
+		)
+	)
+	(wire
+		(pts
 			(xy 91.44 176.53) (xy 91.44 175.26)
 		)
@@
 	(wire
 		(pts
+			(xy 200.66 138.43) (xy 189.23 138.43)
+		)
+		(stroke
+			(width 0)
+			(type default)
+		)
+	)
+	(wire
+		(pts
 			(xy 78.74 173.99) (xy 78.74 175.26)
 		)
@@
 	(wire
 		(pts
-			(xy 189.23 138.43) (xy 200.66 138.43)
+			(xy 180.34 140.97) (xy 200.66 140.97)
 		)
 		(stroke
@@
 	(symbol
 		(lib_id "power:+3.3V")
-		(at 189.23 138.43 0)
+		(at 180.34 140.97 0)
 		(unit 1)
 		(exclude_from_sim no)
@@
 		(fields_autoplaced yes)
 		(property "Reference" "#PWR065"
-			(at 189.23 142.24 0)
+			(at 180.34 144.78 0)
 			(effects
 				(font
@@
 		)
 		(property "Value" "+3.3V"
-			(at 189.23 133.35 0)
+			(at 180.34 135.89 0)
 			(effects
 				(font
@@
 		)
 		(property "Footprint" ""
-			(at 189.23 138.43 0)
+			(at 180.34 140.97 0)
 			(effects
 				(font
@@
 		)
 		(property "Datasheet" ""
-			(at 189.23 138.43 0)
+			(at 180.34 140.97 0)
 			(effects
 				(font
@@
 		)
 		(property "Description" "Power symbol creates a global label with name \"+3.3V\""
-			(at 189.23 138.43 0)
-			(effects
-				(font
+			(at 180.34 140.97 0)
+			(effects
+				(font

Commit message: 22.05.2026
Connections:
- net ADC1: no longer U1.27 (PB13)
- net ADC3: no longer U1.28 (PB14)
- net DISCHARGE1: no longer U1.46 (PB9)
- net DISCHARGE3: no longer U1.26 (PB12)
- net MUX0_IN: now also U1.26 (PB12); no longer U1.11 (PA3)
- net MUX1_IN: now also U1.25 (PB11); no longer U1.10 (PA2)
- net MUX2_IN: now also U1.27 (PB13); no longer U1.32 (PA10)
- net MUX3_IN: now also U1.28 (PB14); no longer U1.31 (PA9)
- net MUX_S0: now also U1.41 (PB4); no longer U1.44 (PB7)
- net MUX_S1: now also U1.39 (PA15); no longer U1.43 (PB6)
- net MUX_S2: now also U1.43 (PB6); no longer U1.42 (PB5)
- net MUX_S3: now also U1.46 (PB9); no longer U1.41 (PB4)
