File: Romashka EC non-matrix/Romashka EC non-matrix.kicad_sch (KiCad schematic)
At the start: 40 parts, among them J1 Daisy40, J2 RS40, J3 JJ40, J4 JSB USB, J5 SOICbite, U1 STM32G474CBTx, U2 USBLC6-2P6, U3 TPS7A2033, Y1 Crystal_GND24_Small

Commit message: 20.08.2026
Parts:
- removed C13: 10uF, Capacitor_SMD:C_0805_2012Metric, symbol Device:C_Small
Connections:
- net MUX_EN: now reaches U1.32 (PA10)
Changed lines of the file:
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@@
 	)
 	(junction
-		(at 91.44 175.26)
-		(diameter 0)
-		(color 0 0 0 0)
-	)
-	(junction
 		(at 24.13 64.77)
 		(diameter 0)
@@
 	(wire
 		(pts
-			(xy 91.44 176.53) (xy 91.44 175.26)
-		)
-		(stroke
-			(width 0)
-			(type default)
-		)
-	)
-	(wire
-		(pts
 			(xy 181.61 30.48) (xy 181.61 29.21)
 		)
@@
 	(wire
 		(pts
-			(xy 91.44 182.88) (xy 91.44 181.61)
-		)
-		(stroke
-			(width 0)
-			(type default)
-		)
-	)
-	(wire
-		(pts
 			(xy 248.92 24.13) (xy 260.35 24.13)
 		)
@@
 		)
 	)
+	(global_label "MUX_EN"
+		(shape input)
+		(at 247.65 66.04 0)
+		(fields_autoplaced yes)
+		(effects
+			(font
+				(size 1.27 1.27)
+			)
+			(justify left)
+		)
+		(property "Intersheetrefs" "${INTERSHEET_REFS}"
+			(at 258.0737 66.04 0)
+			(effects
+				(font
+					(size 1.27 1.27)
+				)
+				(justify left)
+				(hide yes)
+			)
+		)
+	)
 	(global_label "SWDIO"
 		(shape input)
@@
 	)
 	(symbol
-		(lib_id "power:GND")
-		(at 91.44 182.88 0)
-		(unit 1)
-		(exclude_from_sim no)
-		(in_bom yes)
-		(on_board yes)
-		(dnp no)
-		(fields_autoplaced yes)
-		(property "Reference" "#PWR030"
-			(at 91.44 189.23 0)
-			(effects
-				(font
-					(size 1.27 1.27)
-				)
-				(hide yes)
-			)
-		)
-		(property "Value" "GND"
-			(at 91.44 187.96 0)
-			(effects
-				(font
-					(size 1.27 1.27)
-				)
-			)
-		)
-		(property "Footprint" ""
-			(at 91.44 182.88 0)
-			(effects
-				(font
-					(size 1.27 1.27)
-				)
-				(hide yes)
-			)
-		)
-		(property "Datasheet" ""
-			(at 91.44 182.88 0)
-			(effects
-				(font
-					(size 1.27 1.27)
-				)
-				(hide yes)
-			)
-		)
-		(property "Description" "Power symbol creates a global label with name \"GND\" , ground"
-			(at 91.44 182.88 0)
-			(effects
-				(font
-					(size 1.27 1.27)
-				)
-				(hide yes)
-			)
-		)
-		(pin "1"
-		)
-		(instances
-			(project "Romashka EC non-matrix"
-				(path "/69f48e55-4bf1-48a7-a2c4-b2689bdf9720"
-					(reference "#PWR030")
-					(unit 1)
-				)
-			)
-		)
-	)
-	(symbol
 		(lib_id "Device:C_Small")
 		(at 46.99 184.15 180)
@@
 					(unit 1)
 				)
-			)
-		)
-	)
-	(symbol
-		(lib_id "Device:C_Small")
-		(at 91.44 179.07 180)
-		(unit 1)
-		(exclude_from_sim no)
-		(in_bom yes)
-		(on_board yes)
-		(dnp no)
-		(property "Reference" "C13"
-			(at 93.98 177.7935 0)
-			(effects
-				(font
-					(size 1.27 1.27)
-				)
-				(justify right)
-			)
-		)
-		(property "Value" "10uF"
-			(at 93.98 180.3335 0)
-			(effects
-				(font
-					(size 1.27 1.27)
-				)
-				(justify right)
-			)
-		)
-		(property "Footprint" "Capacitor_SMD:C_0805_2012Metric"
-			(at 91.44 179.07 0)
-			(effects
-				(font
-					(size 1.27 1.27)
-				)
-				(hide yes)
-			)
-		)
-		(property "Datasheet" "~"
-			(at 91.44 179.07 0)
-			(effects
-				(font
-					(size 1.27 1.27)
-				)
-				(hide yes)
-			)
-		)
-		(property "Description" "Unpolarized capacitor, small symbol"
-			(at 91.44 179.07 0)
-			(effects
-				(font
-					(size 1.27 1.27)
-				)
-				(hide yes)
-			)
-		)
-		(pin "1"
-		)
-		(pin "2"
-		)
-		(instances
-			(project "Romashka EC non-matrix"
-				(path "/69f48e55-4bf1-48a7-a2c4-b2689bdf9720"
-					(reference "C13")
-					(unit 1)
-				)

Commit message: 21.08.2026
Connections:
- net +3.3V: now also J5.7 (Pin_7); no longer J5.6 (Pin_6)
- net ADC1: now also U1.11 (PA3)
- net ADC3: now also U1.30 (PA8)
- net DISCHARGE1: now also U1.10 (PA2)
- net DISCHARGE2: now also U1.44 (PB7); no longer U1.9 (PA1)
- net DISCHARGE3: now also U1.8 (PA0)
- net GND: now also J5.6 (Pin_6); no longer J5.7 (Pin_7)

Commit message: 23.08.2026
Parts:
- removed BOOT_SW1, RESET_SW1: Omron b3u, Button_Switch_SMD:SW_SPST_B3U-1000P, symbol Switch:SW_DPST_x2
- added SW_BOOT0: MSK12C, FriedSoul_switches:slider-msk12c, symbol Switch:SW_DPDT_x2
Connections:
- net +3.3V: now also SW_BOOT0.1 (A)
- net BOOT0: now also SW_BOOT0.2 (B)
- net DISCHARGE2: now also U1.9 (PA1); no longer U1.44 (PB7)
- net GND: now also SW_BOOT0.3 (C)
Other:
- moved on the sheet: C14, R12
