File: Romashka EC non-matrix/Romashka EC non-matrix.kicad_sch (KiCad schematic)
At the start: 38 parts, among them J1 Daisy40, J2 RS40, J3 JJ40, J4 JSB USB, J5 SOICbite, U1 STM32G474CBTx, U2 USBLC6-2P6, U3 TPS7A2033, Y1 Crystal_GND24_Small

Commit message: 24.08.2026
Connections:
- net ADC1: now also U1.17 (PB1); no longer U1.11 (PA3)
- net ADC2: now also U1.11 (PA3); no longer U1.12 (PA4)
- net ADC3: now also U1.29 (PB15); no longer U1.30 (PA8)
- net DISCHARGE1: now also U1.16 (PB0); no longer U1.10 (PA2)
- net DISCHARGE3: now also U1.27 (PB13); no longer U1.8 (PA0)
- net MUX2_IN: now also U1.31 (PA9); no longer U1.27 (PB13)
- net MUX3_IN: now also U1.30 (PA8); no longer U1.28 (PB14)
Changed lines of the file:
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@@
 	(global_label "DISCHARGE3"
 		(shape input)
-		(at 247.65 40.64 0)
-		(fields_autoplaced yes)
-		(effects
-			(font
-				(size 1.27 1.27)
-			)
-			(justify left)
-		)
-		(property "Intersheetrefs" "${INTERSHEET_REFS}"
-			(at 262.3071 40.64 0)
-			(effects
-				(font
-					(size 1.27 1.27)
-				)
-				(justify left)
+		(at 212.09 101.6 180)
+		(fields_autoplaced yes)
+		(effects
+			(font
+				(size 1.27 1.27)
+			)
+			(justify right)
+		)
+		(property "Intersheetrefs" "${INTERSHEET_REFS}"
+			(at 197.4329 101.6 0)
+			(effects
+				(font
+					(size 1.27 1.27)
+				)
+				(justify right)
 				(hide yes)
 			)
@@
 	(global_label "DISCHARGE1"
 		(shape input)
-		(at 247.65 45.72 0)
-		(fields_autoplaced yes)
-		(effects
-			(font
-				(size 1.27 1.27)
-			)
-			(justify left)
-		)
-		(property "Intersheetrefs" "${INTERSHEET_REFS}"
-			(at 262.3071 45.72 0)
-			(effects
-				(font
-					(size 1.27 1.27)
-				)
-				(justify left)
+		(at 212.09 68.58 180)
+		(fields_autoplaced yes)
+		(effects
+			(font
+				(size 1.27 1.27)
+			)
+			(justify right)
+		)
+		(property "Intersheetrefs" "${INTERSHEET_REFS}"
+			(at 197.4329 68.58 0)
+			(effects
+				(font
+					(size 1.27 1.27)
+				)
+				(justify right)
 				(hide yes)
 			)
@@
 	(global_label "ADC2"
 		(shape input)
-		(at 247.65 50.8 0)
-		(fields_autoplaced yes)
-		(effects
-			(font
-				(size 1.27 1.27)
-			)
-			(justify left)
-		)
-		(property "Intersheetrefs" "${INTERSHEET_REFS}"
-			(at 255.4733 50.8 0)
+		(at 247.65 48.26 0)
+		(fields_autoplaced yes)
+		(effects
+			(font
+				(size 1.27 1.27)
+			)
+			(justify left)
+		)
+		(property "Intersheetrefs" "${INTERSHEET_REFS}"
+			(at 255.4733 48.26 0)
 			(effects
 				(font
@@
 	(global_label "MUX2_IN"
 		(shape input)
-		(at 212.09 101.6 180)
-		(fields_autoplaced yes)
-		(effects
-			(font
-				(size 1.27 1.27)
-			)
-			(justify right)
-		)
-		(property "Intersheetrefs" "${INTERSHEET_REFS}"
-			(at 201.001 101.6 0)
-			(effects
-				(font
-					(size 1.27 1.27)
-				)
-				(justify right)
+		(at 247.65 63.5 0)
+		(fields_autoplaced yes)
+		(effects
+			(font
+				(size 1.27 1.27)
+			)
+			(justify left)
+		)
+		(property "Intersheetrefs" "${INTERSHEET_REFS}"
+			(at 258.739 63.5 0)
+			(effects
+				(font
+					(size 1.27 1.27)
+				)
+				(justify left)
 				(hide yes)
 			)
@@
 	(global_label "ADC1"
 		(shape input)
-		(at 247.65 48.26 0)
-		(fields_autoplaced yes)
-		(effects
-			(font
-				(size 1.27 1.27)
-			)
-			(justify left)
-		)
-		(property "Intersheetrefs" "${INTERSHEET_REFS}"
-			(at 255.4733 48.26 0)
-			(effects
-				(font
-					(size 1.27 1.27)
-				)
-				(justify left)
+		(at 212.09 71.12 180)
+		(fields_autoplaced yes)
+		(effects
+			(font
+				(size 1.27 1.27)
+			)
+			(justify right)
+		)
+		(property "Intersheetrefs" "${INTERSHEET_REFS}"
+			(at 204.2667 71.12 0)
+			(effects
+				(font
+					(size 1.27 1.27)
+				)
+				(justify right)
 				(hide yes)
 			)
@@
 	(global_label "MUX3_IN"
 		(shape input)
-		(at 212.09 104.14 180)
-		(fields_autoplaced yes)
-		(effects
-			(font
-				(size 1.27 1.27)
-			)
-			(justify right)
-		)
-		(property "Intersheetrefs" "${INTERSHEET_REFS}"
-			(at 201.001 104.14 0)
-			(effects
-				(font
-					(size 1.27 1.27)
-				)
-				(justify right)
+		(at 247.65 60.96 0)
+		(fields_autoplaced yes)
+		(effects
+			(font
+				(size 1.27 1.27)
+			)
+			(justify left)
+		)
+		(property "Intersheetrefs" "${INTERSHEET_REFS}"
+			(at 258.739 60.96 0)
+			(effects
+				(font
+					(size 1.27 1.27)
+				)
+				(justify left)
 				(hide yes)
 			)
@@
 	(global_label "ADC3"
 		(shape input)
-		(at 247.65 60.96 0)
-		(fields_autoplaced yes)
-		(effects
-			(font
-				(size 1.27 1.27)
-			)
-			(justify left)
-		)
-		(property "Intersheetrefs" "${INTERSHEET_REFS}"
-			(at 255.4733 60.96 0)
-			(effects
-				(font
-					(size 1.27 1.27)
-				)
-				(justify left)
-				(hide yes)
-			)
+		(at 212.09 106.68 180)
+		(fields_autoplaced yes)
+		(effects
+			(font
+				(size 1.27 1.27)
+			)
+			(justify right)
+		)
+		(property "Intersheetrefs" "${INTERSHEET_REFS}"
+			(at 204.2667 106.68 0)
+			(effects
+				(font
+					(size 1.27 1.27)
+				)
+				(justify right)
+				(hide yes)
+			)

Commit message: 25.08.2026
Parts:
- added H10, H7, H8, H9: MountingHole, FriesSoul_misc:m2 hole, symbol Mechanical:MountingHole
- H1, H2, H3, H4, H5, H6: footprint Kicad footprints:m2 hole -> FriesSoul_misc:m2 hole
- J5: footprint Kicad footprints:SOICbite_footprint -> FriesSoul_misc:SOICbite_footprint
Connections:
- net ADC0: now also U1.11 (PA3); no longer U1.14 (PA6)
- net ADC1: now also U1.14 (PA6); no longer U1.17 (PB1)
- net ADC2: now also U1.17 (PB1); no longer U1.11 (PA3)
- net DISCHARGE0: now also U1.9 (PA1); no longer U1.13 (PA5)
- net DISCHARGE1: now also U1.13 (PA5); no longer U1.16 (PB0)
- net DISCHARGE2: now also U1.16 (PB0); no longer U1.9 (PA1)
