File: Romashka EC non-matrix/Romashka EC non-matrix.kicad_pcb (KiCad board)
At the start: 2 copper layers, 228.6 x 76.2 mm, 145 parts, among them J1 Daisy40, J2 RS40, J3 JJ40, J4 JSB USB, J5 SOICbite, SW1 EC_SW, SW10 EC_SW, SW11 EC_SW, SW12 EC_SW, SW13 EC_SW, SW14 EC_SW, SW15 EC_SW, SW16 EC_SW, SW17 EC_SW, SW18 EC_SW, SW19 EC_SW, SW2 EC_SW, SW20 EC_SW, SW21 EC_SW, SW22 EC_SW, SW23 EC_SW, SW24 EC_SW, SW25 EC_SW, SW26 EC_SW, SW27 EC_SW, SW28 EC_SW, SW29 EC_SW, SW3 EC_SW, SW30 EC_SW, SW31 EC_SW, SW32 EC_SW, SW35 EC_SW, SW36 EC_SW, SW38 EC_SW, SW39 EC_SW, SW4 EC_SW, SW40 EC_SW, SW42 EC_SW, SW43 EC_SW, SW44 EC_SW, SW45 EC_SW, SW47 EC_SW, SW49 EC_SW, SW5 EC_SW, SW6 EC_SW, SW7 EC_SW, SW8 EC_SW, SW9 EC_SW, U1 STM32G474CBTx, U10 TLV9061xDBV, U11 TLV9061xDBV, U12 TLV9061xDBV, U13 TLV9061xDBV, U14 TLV9061xDBV, U15 TLV9061xDBV, U2 USBLC6-2P6, U3 TPS7A2033, U4 4051, U5 4051, U6 4051, U7 4051, U8 4051, U9 4051

Commit message: 24.04.2026
Parts:
- removed the C13 at (186.1, 48.8)
- removed the C14 at (223.8, 69.8)
- removed the C22 at (175.6, 113.4)
- removed the C24 at (175.6, 118.4)
- removed C26, C28, C30, C32: 1uF, Capacitor_SMD:C_0603_1608Metric
- removed C29, C31: 470pF, Capacitor_SMD:C_0603_1608Metric
- removed C36, C37: 100nF, Capacitor_SMD:C_0402_1005Metric
- removed the R19 at (169.5, 87.3)
- removed the R20 at (172.6, 87.3)
- removed the R25 at (196.8, 62.3)
- removed the R26 at (173.8, 84.5)
- removed U14, U15: TLV9061xDBV, Package_TO_SOT_SMD:SOT-23-5
- removed the U8 at (189.3, 48.8)
- removed the U9 at (220.7, 69.8)
- added R10: 100K, Resistor_SMD:R_0603_1608Metric, B.Cu at (176.0, 115.5)
- added R13: 100K, Resistor_SMD:R_0603_1608Metric, B.Cu at (176.0, 118.0)
- added R14: 100K, Resistor_SMD:R_0603_1608Metric, B.Cu at (176.0, 120.5)
- added R15: 100K, Resistor_SMD:R_0603_1608Metric, B.Cu at (176.0, 123.0)
- added R16: 100K, Resistor_SMD:R_0603_1608Metric, B.Cu at (176.0, 125.5)
- added R21: 100K, Resistor_SMD:R_0603_1608Metric, B.Cu at (176.0, 133.1)
- added R22: 100K, Resistor_SMD:R_0603_1608Metric, B.Cu at (172.0, 108.0)
- added R23: 100K, Resistor_SMD:R_0603_1608Metric, B.Cu at (172.0, 110.5)
- added R24: 100K, Resistor_SMD:R_0603_1608Metric, B.Cu at (172.0, 113.0)
- added R29: 100K, Resistor_SMD:R_0603_1608Metric, B.Cu at (172.0, 115.5)
- added R30: 100K, Resistor_SMD:R_0603_1608Metric, B.Cu at (172.0, 118.0)
- added R33: 100K, Resistor_SMD:R_0603_1608Metric, B.Cu at (172.0, 120.5)
- added R34: 100K, Resistor_SMD:R_0603_1608Metric, B.Cu at (172.0, 123.0)
- added R35: 100K, Resistor_SMD:R_0603_1608Metric, B.Cu at (172.0, 125.5)
- added R36: 100K, Resistor_SMD:R_0603_1608Metric, B.Cu at (172.0, 128.0)
- added R37: 100K, Resistor_SMD:R_0603_1608Metric, B.Cu at (172.0, 130.5)
- added R38: 100K, Resistor_SMD:R_0603_1608Metric, B.Cu at (172.0, 133.1)
- added R39: 100K, Resistor_SMD:R_0603_1608Metric, B.Cu at (168.0, 108.0)
- added R40: 100K, Resistor_SMD:R_0603_1608Metric, B.Cu at (168.0, 110.5)
- added R41: 100K, Resistor_SMD:R_0603_1608Metric, B.Cu at (168.0, 113.0)
- added R42: 100K, Resistor_SMD:R_0603_1608Metric, B.Cu at (168.0, 115.5)
- added R43: 100K, Resistor_SMD:R_0603_1608Metric, B.Cu at (168.0, 118.0)
- added R44: 100K, Resistor_SMD:R_0603_1608Metric, B.Cu at (168.0, 120.5)
- added R45: 100K, Resistor_SMD:R_0603_1608Metric, B.Cu at (168.0, 123.0)
- added R46: 100K, Resistor_SMD:R_0603_1608Metric, B.Cu at (168.0, 125.5)
- added R47: 100K, Resistor_SMD:R_0603_1608Metric, B.Cu at (168.0, 128.0)
- added R48: 100K, Resistor_SMD:R_0603_1608Metric, B.Cu at (168.0, 130.5)
- added R49: 100K, Resistor_SMD:R_0603_1608Metric, B.Cu at (168.0, 133.1)
- added R50: 100K, Resistor_SMD:R_0603_1608Metric, B.Cu at (164.0, 108.0)
- added R51: 100K, Resistor_SMD:R_0603_1608Metric, B.Cu at (164.0, 110.5)
- added R52: 100K, Resistor_SMD:R_0603_1608Metric, B.Cu at (164.0, 113.0)
- added R53: 100K, Resistor_SMD:R_0603_1608Metric, B.Cu at (164.0, 115.5)
- added R54: 100K, Resistor_SMD:R_0603_1608Metric, B.Cu at (164.0, 118.0)
- added R55: 100K, Resistor_SMD:R_0603_1608Metric, B.Cu at (164.0, 120.5)
- added R56: 100K, Resistor_SMD:R_0603_1608Metric, B.Cu at (164.0, 123.0)
- added R57: 100K, Resistor_SMD:R_0603_1608Metric, B.Cu at (164.0, 125.5)
- added R58: 100K, Resistor_SMD:R_0603_1608Metric, B.Cu at (164.0, 128.0)
- added R59: 100K, Resistor_SMD:R_0603_1608Metric, B.Cu at (164.0, 130.5)
- added R60: 100K, Resistor_SMD:R_0603_1608Metric, B.Cu at (164.0, 133.1)
- added R61: 100K, Resistor_SMD:R_0603_1608Metric, B.Cu at (160.0, 108.0)
- added R62: 100K, Resistor_SMD:R_0603_1608Metric, B.Cu at (160.0, 110.5)
- added R63: 100K, Resistor_SMD:R_0603_1608Metric, B.Cu at (160.0, 113.0)
- added R64: 100K, Resistor_SMD:R_0603_1608Metric, B.Cu at (160.0, 115.5)
- added R65: 100K, Resistor_SMD:R_0603_1608Metric, B.Cu at (160.0, 118.0)
- added R66: 100K, Resistor_SMD:R_0603_1608Metric, B.Cu at (160.0, 120.5)
- added R67: 100K, Resistor_SMD:R_0603_1608Metric, B.Cu at (160.0, 123.0)
- added R68: 100K, Resistor_SMD:R_0603_1608Metric, B.Cu at (160.0, 125.5)
- added R69: 100K, Resistor_SMD:R_0603_1608Metric, B.Cu at (160.0, 128.0)
- added R7: 100K, Resistor_SMD:R_0603_1608Metric, B.Cu at (176.0, 108.0)
- added R70: 100K, Resistor_SMD:R_0603_1608Metric, B.Cu at (160.0, 130.5)
- added R71: 100K, Resistor_SMD:R_0603_1608Metric, B.Cu at (160.0, 133.1)
- added R72: 100K, Resistor_SMD:R_0603_1608Metric, B.Cu at (156.0, 108.0)
- added R73: 100K, Resistor_SMD:R_0603_1608Metric, B.Cu at (156.0, 110.5)
- added R74: 100K, Resistor_SMD:R_0603_1608Metric, B.Cu at (156.0, 113.0)
- added R75: 100K, Resistor_SMD:R_0603_1608Metric, B.Cu at (156.0, 115.5)
- added R76: 100K, Resistor_SMD:R_0603_1608Metric, B.Cu at (156.0, 118.0)
- added R77: 100K, Resistor_SMD:R_0603_1608Metric, B.Cu at (156.0, 120.5)
- added R78: 100K, Resistor_SMD:R_0603_1608Metric, B.Cu at (156.0, 123.0)
- added R79: 100K, Resistor_SMD:R_0603_1608Metric, B.Cu at (156.0, 125.5)
- added R8: 100K, Resistor_SMD:R_0603_1608Metric, B.Cu at (176.0, 110.5)
- added R80: 100K, Resistor_SMD:R_0603_1608Metric, B.Cu at (156.0, 128.0)
- added R9: 100K, Resistor_SMD:R_0603_1608Metric, B.Cu at (176.0, 113.0)
- R17: value 33K -> 100K
- R18: value 330 -> 100K
- SW14, SW15, SW16, SW17, SW18, SW20, SW21, SW22, SW32: footprint Kicad footprints:ecs_pad_1U_hybrid_hotswap_V3_switched_sides -> Kicad footprints:ecs_pad_1U_hybrid_hotswap_V3
- SW23, SW24, SW29, SW39, SW40: footprint Kicad footprints:ecs_pad_1U_hybrid_hotswap_V3 -> Kicad footprints:ecs_pad_1U_hybrid_hotswap_V3_switched_sides
- U4, U5, U6, U7: value 4051 -> HEF4067BTT; footprint Package_SO:Texas_DYY0016A_TSOT-23-16_2x4.2mm_P0.5mm -> Package_SO:TSSOP-24_4.4x7.8mm_P0.65mm
- moved R19 136.4 mm to (24.6, 14.3)
- moved R2 131.7 mm to (43.7, 14.3)
- moved R20 128.4 mm to (38.9, 14.3), turned to 0 degrees
- moved R4 112.6 mm to (57.9, 14.3), turned to 0 degrees
- moved C17 109.1 mm to (149.2, 29.8), turned to -90 degrees
- moved U3 104.8 mm to (146.1, 29.8), turned to 0 degrees
- moved R1 99.6 mm to (119.9, 14.3)
- moved C11 98.3 mm to (130.2, 122.7), turned to -90 degrees
- moved C12 96.0 mm to (132.6, 122.6), turned to -90 degrees
- moved R3 89.9 mm to (134.1, 14.3), turned to 0 degrees
- moved C10 83.7 mm to (131.4, 122.6), turned to -90 degrees
- moved R81 82.5 mm to (221.1, 29.4), turned to 0 degrees
- moved U5 82.2 mm to (161.6, 96.0), turned to 180 degrees
- moved R88 82.1 mm to (222.6, 31.8), turned to -90 degrees
- moved C16 80.4 mm to (143.3, 29.8), turned to -90 degrees
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- renumbered C15 to C13, C16 to C14, C17 to C15, C18 to C16, C19 to C17, C20 to C18, C35 to C19, C33 to C20, C34 to C21, C21 to C22, C27 to C23, C23 to C24, J5 to J4, J4 to J5, R29 to R11, R30 to R12, R5 to R19, R6 to R20, R33 to R25, R34 to R26, R35 to R27, R36 to R28, R11 to R31, R12 to R32, R27 to R5, R28 to R6, R21 to R81, R24 to R82, R22 to R83, R23 to R84, R7 to R85, R15 to R86, R9 to R87, R8 to R88, R13 to R89, R16 to R90, R10 to R91, R14 to R92, U11 to U10, U12 to U11, U10 to U8, U13 to U9
Connections:
- C22 pad 1: DISCHAEGE0 -> DISCHARGE0
- C23 pad 1: DISCHAEGE3 -> DISCHARGE3
- C24 pad 1: DISCHAEGE1 -> DISCHARGE1
- C25 pad 1: DISCHAEGE2 -> DISCHARGE2
- R11 pad 1: unconnected-(R29-Pad1) -> Net-(U1-PA2)
- R12 pad 1: unconnected-(R30-Pad1) -> Net-(U1-PA3)
- R17 pad 1: Net-(U14--) -> GND
- R17 pad 2: ADC4 -> MUX0_D4
- R18 pad 1: Net-(U14--) -> GND
- R18 pad 2: GND -> MUX2_D1
- R25 pad 2: unconnected-(R33-Pad2) -> Net-(U1-PB12)
- R26 pad 2: unconnected-(R34-Pad2) -> Net-(U1-PB13)
- R27 pad 2: unconnected-(R35-Pad2) -> Net-(U1-PB14)
- R28 pad 2: unconnected-(R36-Pad2) -> Net-(U1-PB15)
- R5 pad 1: unconnected-(R27-Pad1) -> Net-(U1-PA0)
- R6 pad 1: unconnected-(R28-Pad1) -> Net-(U1-PA1)
- R81 pad 1: DISCHAEGE0 -> DISCHARGE0
- R82 pad 2: DISCHAEGE3 -> DISCHARGE3
- R83 pad 1: DISCHAEGE1 -> DISCHARGE1
- R84 pad 2: DISCHAEGE2 -> DISCHARGE2
- SW10 pad 1: SENSE4 -> SENSE0
- SW11 pad 1: SENSE5 -> SENSE0
- SW12 pad 1: SENSE5 -> SENSE0
- SW13 pad 1: SENSE0 -> SENSE1
- SW13 pad 2: MUX0_D5 -> unconnected-(SW13-Pad2)
- SW15 pad 1: SENSE2 -> SENSE1
- SW16 pad 1: SENSE2 -> SENSE1
- SW17 pad 1: SENSE2 -> SENSE1
- SW18 pad 1: SENSE2 -> SENSE1
- SW19 pad 1: SENSE2 -> SENSE1
- SW2 pad 1: SENSE1 -> SENSE0
- SW20 pad 1: SENSE3 -> SENSE1
- SW21 pad 1: SENSE4 -> SENSE1
- SW22 pad 1: SENSE4 -> SENSE1
- SW23 pad 1: SENSE5 -> SENSE0
- SW24 pad 1: SENSE0 -> SENSE2
- SW24 pad 2: MUX0_D7 -> unconnected-(SW24-Pad2)
- SW25 pad 1: SENSE1 -> SENSE2
- SW26 pad 1: SENSE1 -> SENSE2
- SW27 pad 1: SENSE1 -> SENSE2
- SW28 pad 1: SENSE1 -> SENSE2
- SW29 pad 1: SENSE1 -> SENSE2
- SW3 pad 1: SENSE2 -> SENSE0
- SW31 pad 1: SENSE3 -> SENSE2
- SW32 pad 1: SENSE4 -> SENSE2
- SW35 pad 1: SENSE0 -> SENSE2
- SW35 pad 2: MUX0_D6 -> unconnected-(SW35-Pad2)
- SW36 pad 1: SENSE0 -> SENSE3
- SW36 pad 2: MUX0_D4 -> unconnected-(SW36-Pad2)
- SW38 pad 1: SENSE0 -> SENSE3
- SW38 pad 2: MUX0_D1 -> unconnected-(SW38-Pad2)
- SW39 pad 1: SENSE0 -> SENSE3
- SW39 pad 2: MUX0_D3 -> unconnected-(SW39-Pad2)
- SW4 pad 1: SENSE3 -> SENSE0
- SW40 pad 1: SENSE5 -> SENSE3
- SW42 pad 1: SENSE5 -> SENSE3
- SW43 pad 1: SENSE4 -> SENSE3
- SW44 pad 1: SENSE5 -> SENSE3
- SW45 pad 1: SENSE0 -> SENSE3
- SW45 pad 2: MUX0_D2 -> unconnected-(SW45-Pad2)
- SW47 pad 1: SENSE5 -> SENSE3
- SW49 pad 1: SENSE0 -> SENSE3
- SW49 pad 2: MUX0_D0 -> unconnected-(SW49-Pad2)
- SW5 pad 1: SENSE3 -> SENSE0
- SW6 pad 1: SENSE3 -> SENSE0
- SW7 pad 1: SENSE3 -> SENSE0
- SW8 pad 1: SENSE3 -> SENSE0
- SW9 pad 1: SENSE4 -> SENSE0
- U1 pad 10: unconnected-(U1-PA2-Pad10) -> Net-(U1-PA2)
- U1 pad 11: unconnected-(U1-PA3-Pad11) -> Net-(U1-PA3)
- U1 pad 12: unconnected-(U1-PA4-Pad12) -> DISCHARGE3
- U1 pad 13: unconnected-(U1-PA5-Pad13) -> DISCHARGE2
- U1 pad 14: unconnected-(U1-PA6-Pad14) -> DISCHARGE1
- U1 pad 15: unconnected-(U1-PA7-Pad15) -> DISCHARGE0
- U1 pad 26: unconnected-(U1-PB12-Pad26) -> Net-(U1-PB12)
- U1 pad 27: unconnected-(U1-PB13-Pad27) -> Net-(U1-PB13)
- U1 pad 28: unconnected-(U1-PB14-Pad28) -> Net-(U1-PB14)
- U1 pad 29: unconnected-(U1-PB15-Pad29) -> Net-(U1-PB15)
- U1 pad 41: MUX_S2 -> MUX_S3
- U1 pad 42: MUX_S1 -> MUX_S2
- U1 pad 43: MUX_S0 -> MUX_S1
- U1 pad 44: unconnected-(U1-PB7-Pad44) -> MUX_S0
- U1 pad 8: unconnected-(U1-PA0-Pad8) -> Net-(U1-PA0)
- U1 pad 9: unconnected-(U1-PA1-Pad9) -> Net-(U1-PA1)
- U10 pad 3: DISCHAEGE1 -> DISCHARGE1
- U11 pad 3: DISCHAEGE2 -> DISCHARGE2
- U4 pad 1: MUX0_D4 -> MUX0_IN
- U4 pad 10: MUX_S1 -> MUX_S0
- U4 pad 11: MUX_S0 -> MUX_S1
- U4 pad 12: MUX0_D3 -> GND
- U4 pad 13: MUX0_D0 -> MUX_S3
- U4 pad 14: MUX0_D1 -> MUX_S2
- U4 pad 15: MUX0_D2 -> GND
- U4 pad 16: +3.3VA -> MUX0_D15
- U4 pad 2: MUX0_D6 -> MUX0_D7
- U4 pad 3: MUX0_IN -> MUX0_D6
- U4 pad 4: MUX0_D7 -> MUX0_D5
- U4 pad 5: MUX0_D5 -> MUX0_D4
- U4 pad 6: MUX0_EN -> MUX0_D3
- U4 pad 7: GND -> MUX0_D2
- U4 pad 8: GND -> MUX0_D1
- U4 pad 9: MUX_S2 -> MUX0_D0
- U5 pad 1: MUX1_D4 -> MUX0_IN
- U5 pad 10: MUX_S1 -> MUX_S0
- U5 pad 11: MUX_S0 -> MUX_S1
- U5 pad 12: MUX1_D3 -> GND
- U5 pad 13: MUX1_D0 -> MUX_S3
- U5 pad 14: MUX1_D1 -> MUX_S2
- U5 pad 15: MUX1_D2 -> GND
- U5 pad 16: +3.3VA -> MUX1_D15
- U5 pad 2: MUX1_D6 -> MUX1_D7
- U5 pad 3: MUX1_IN -> MUX1_D6
- U5 pad 4: MUX1_D7 -> MUX1_D5
- U5 pad 5: MUX1_D5 -> MUX1_D4
- U5 pad 6: MUX1_EN -> MUX1_D3
- U5 pad 7: GND -> MUX1_D2
- U5 pad 8: GND -> MUX1_D1
- U5 pad 9: MUX_S2 -> MUX1_D0
- U6 pad 1: MUX2_D4 -> MUX0_IN
- U6 pad 10: MUX_S1 -> MUX_S0
- U6 pad 11: MUX_S0 -> MUX_S1
- U6 pad 12: MUX2_D3 -> GND
- U6 pad 13: MUX2_D0 -> MUX_S3
- U6 pad 14: MUX2_D1 -> MUX_S2
- U6 pad 15: MUX2_D2 -> GND
- U6 pad 16: +3.3VA -> MUX2_D15
- U6 pad 2: MUX2_D6 -> MUX2_D7
- U6 pad 3: MUX2_IN -> MUX2_D6
- U6 pad 4: MUX2_D7 -> MUX2_D5
- U6 pad 5: MUX2_D5 -> MUX2_D4
- U6 pad 6: MUX2_EN -> MUX2_D3
- U6 pad 7: GND -> MUX2_D2
- U6 pad 8: GND -> MUX2_D1
- U6 pad 9: MUX_S2 -> MUX2_D0
- U7 pad 1: MUX3_D4 -> MUX0_IN
- U7 pad 10: MUX_S1 -> MUX_S0
- U7 pad 11: MUX_S0 -> MUX_S1
- U7 pad 12: MUX3_D3 -> GND
- U7 pad 13: MUX3_D0 -> MUX_S3
- U7 pad 14: MUX3_D1 -> MUX_S2
- U7 pad 15: MUX3_D2 -> GND
- U7 pad 16: +3.3VA -> MUX3_D15
- U7 pad 2: MUX3_D6 -> MUX3_D7
- U7 pad 3: MUX3_IN -> MUX3_D6
- U7 pad 4: MUX3_D7 -> MUX3_D5
- U7 pad 5: MUX3_D5 -> MUX3_D4
- U7 pad 6: MUX3_EN -> MUX3_D3
- U7 pad 7: GND -> MUX3_D2
- U7 pad 8: GND -> MUX3_D1
- U7 pad 9: MUX_S2 -> MUX3_D0
- U8 pad 3: DISCHAEGE0 -> DISCHARGE0
- U9 pad 3: DISCHAEGE3 -> DISCHARGE3
Routing:
- net SENSE5: track 152.6 -> 0.00 mm, vias 1 -> 0
- net +5V_USB: track 0.00 -> 145.6 mm, vias 0 -> 9
- net DM_USB: track 0.00 -> 144.4 mm, vias 0 -> 3
- net DP_USB: track 0.00 -> 141.2 mm, vias 0 -> 3
- net SENSE3: track 117.8 -> 239.1 mm
- net MUX0_D5: track 116.8 -> 0.00 mm
- net MUX0_D6: track 108.3 -> 0.00 mm
- net SENSE4: track 99.8 -> 0.00 mm, vias 1 -> 0
- net MUX0_D7: track 97.2 -> 0.00 mm
- net SENSE2: track 114.5 -> 202.9 mm
- net MUX0_D4: track 85.0 -> 0.00 mm
- net SENSE0: track 155.1 -> 235.1 mm, vias 1 -> 0
- net MUX0_D2: track 72.3 -> 0.00 mm
- net +3.3V: track 0.00 -> 56.7 mm, vias 0 -> 4
- net D-: track 0.00 -> 52.1 mm
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
Commit message: 27.04.2026
Parts:
- added REF**: m2 hole, Kicad footprints:m2 hole, F.Cu at (127.0, 69.8)
- added REF**: m2 hole, Kicad footprints:m2 hole, F.Cu at (31.8, 69.8)
- added REF**: m2 hole, Kicad footprints:m2 hole, F.Cu at (127.0, 31.8)
- added REF**: m2 hole, Kicad footprints:m2 hole, F.Cu at (31.8, 31.8)
- added REF**: m2 hole, Kicad footprints:m2 hole, F.Cu at (222.2, 69.8)
- added REF**: m2 hole, Kicad footprints:m2 hole, F.Cu at (222.2, 31.8)
- SW1, SW2, SW3, SW35, SW38, SW39: footprint Kicad footprints:ecs_pad_1U_hybrid_hotswap_V3_switched_sides -> Kicad footprints:ecs_pad_1U_hybrid_hotswap_V3
- SW10, SW11, SW12, SW18, SW19, SW20, SW21, SW22, SW32, SW4, SW5: footprint Kicad footprints:ecs_pad_1U_hybrid_hotswap_V3 -> Kicad footprints:ecs_pad_1U_hybrid_hotswap_V3_switched_sides
- moved C24 72.4 mm to (119.9, 63.5), turned to -90 degrees
- moved U10 69.7 mm to (122.6, 63.1), turned to 90 degrees
- moved R83 68.5 mm to (120.3, 60.3), turned to 90 degrees
- moved R87 66.5 mm to (122.6, 60.3), turned to 0 degrees
- moved C20 65.9 mm to (124.6, 61.1), turned to -90 degrees
- moved R91 65.3 mm to (121.8, 57.9)
- moved U6 61.7 mm to (112.7, 48.8)
- moved C6 53.7 mm to (163.1, 76.2)
- moved C5 53.7 mm to (165.5, 74.6)
- moved C7 53.7 mm to (163.1, 77.4)
- moved C8 53.7 mm to (163.5, 73.8)
- moved C1 53.7 mm to (176.3, 83.5)
- moved C2 53.7 mm to (173.8, 84.3)
- moved C3 53.7 mm to (175.8, 81.6)
- moved C4 53.7 mm to (173.8, 74.2)
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Connections:
- SW10 pad 1: SENSE0 -> SENSE3
- SW11 pad 1: SENSE0 -> SENSE3
- SW12 pad 1: SENSE0 -> SENSE3
- SW18 pad 1: SENSE1 -> SENSE2
- SW19 pad 1: SENSE1 -> SENSE2
- SW2 pad 1: SENSE0 -> SENSE1
- SW20 pad 1: SENSE1 -> SENSE2
- SW21 pad 1: SENSE1 -> SENSE2
- SW22 pad 1: SENSE1 -> SENSE3
- SW23 pad 1: SENSE0 -> SENSE3
- SW24 pad 1: SENSE2 -> SENSE0
- SW25 pad 1: SENSE2 -> SENSE0
- SW26 pad 1: SENSE2 -> SENSE0
- SW27 pad 1: SENSE2 -> SENSE0
- SW28 pad 1: SENSE2 -> SENSE1
- SW3 pad 1: SENSE0 -> SENSE1
- SW32 pad 1: SENSE2 -> SENSE3
- SW35 pad 1: SENSE2 -> SENSE0
- SW36 pad 1: SENSE3 -> SENSE0
- SW38 pad 1: SENSE3 -> SENSE0
- SW39 pad 1: SENSE3 -> SENSE0
- SW4 pad 1: SENSE0 -> SENSE1
- SW45 pad 1: SENSE3 -> SENSE0
- SW49 pad 1: SENSE3 -> SENSE0
- SW5 pad 1: SENSE0 -> SENSE1
- SW6 pad 1: SENSE0 -> SENSE2
- SW7 pad 1: SENSE0 -> SENSE2
- SW8 pad 1: SENSE0 -> SENSE2
- SW9 pad 1: SENSE0 -> SENSE2
Routing:
- net +5V_USB: track 145.6 -> 0.00 mm, vias 9 -> 0
- net DM_USB: track 144.4 -> 0.00 mm, vias 3 -> 0
- net DP_USB: track 141.2 -> 0.00 mm, vias 3 -> 0
- net SENSE0: track 235.1 -> 141.3 mm
- net SENSE1: track 155.7 -> 218.9 mm, vias 1 -> 0
- net +3.3V: track 56.7 -> 0.00 mm, vias 4 -> 0
- net D-: track 52.1 -> 0.00 mm
- net D+: track 52.1 -> 0.00 mm
- net SENSE2: track 202.9 -> 154.9 mm, vias 1 -> 0
- net +5V: track 19.5 -> 0.00 mm
- net SENSE3: track 239.1 -> 223.8 mm, vias 1 -> 0
- net +3.3VA: track 12.8 -> 1.90 mm, vias 4 -> 1
- net Net-(J1-CC1): track 10.0 -> 0.00 mm
- net Net-(J1-CC2): track 9.56 -> 0.00 mm
- net unconnected-(SW32-Pad2): track 7.29 -> 0.00 mm
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
Commit message: 28.04.2026
Parts:
- added G***: LOGO, Kicad footprints:Romashka, F.Cu at (167.8, 79.9)
- SW18, SW19, SW20, SW21, SW40, SW42, SW6, SW7: footprint Kicad footprints:ecs_pad_1U_hybrid_hotswap_V3_switched_sides -> Kicad footprints:ecs_pad_1U_hybrid_hotswap_V3
- SW8, SW9: footprint Kicad footprints:ecs_pad_1U_hybrid_hotswap_V3 -> Kicad footprints:ecs_pad_1U_hybrid_hotswap_V3_switched_sides
- moved C12 109.7 mm to (209.2, 44.1), turned to 0 degrees
- moved C10 107.3 mm to (86.9, 25.0), turned to 0 degrees
- moved J5 104.8 mm to (152.0, 31.4), turned to 90 degrees
- moved RESET_SW1 102.7 mm to (201.2, 68.3), turned to 90 degrees
- moved BOOT_SW1 97.3 mm to (197.6, 68.3), turned to -90 degrees
- moved C11 81.2 mm to (148.8, 43.7), turned to 0 degrees
- moved R90 80.4 mm to (164.7, 86.5), turned to 0 degrees
- moved U7 79.3 mm to (211.5, 48.8)
- moved R86 78.5 mm to (163.9, 83.7), turned to 90 degrees
- moved R81 75.5 mm to (158.0, 82.5), turned to 180 degrees
- moved C19 75.4 mm to (164.7, 81.8), turned to 0 degrees
- moved C23 74.8 mm to (167.9, 86.5)
- moved R88 74.8 mm to (156.4, 80.2), turned to 90 degrees
- moved R82 74.6 mm to (171.0, 86.5)
- moved U9 73.5 mm to (166.7, 83.7), turned to 180 degrees
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Connections:
- C10 pad 1: +3.3VA -> +3.3V
- C11 pad 1: +3.3VA -> +3.3V
- C12 pad 1: +3.3VA -> +3.3V
- C9 pad 1: +3.3VA -> +3.3V
- R11 pad 1: Net-(U1-PA2) -> unconnected-(R11-Pad1)
- R12 pad 1: Net-(U1-PA3) -> unconnected-(R12-Pad1)
- R25 pad 2: Net-(U1-PB12) -> unconnected-(R25-Pad2)
- R26 pad 2: Net-(U1-PB13) -> unconnected-(R26-Pad2)
- R27 pad 2: Net-(U1-PB14) -> unconnected-(R27-Pad2)
- R28 pad 2: Net-(U1-PB15) -> unconnected-(R28-Pad2)
- R5 pad 1: Net-(U1-PA0) -> unconnected-(R5-Pad1)
- R6 pad 1: Net-(U1-PA1) -> unconnected-(R6-Pad1)
- U1 pad 10: Net-(U1-PA2) -> unconnected-(U1-PA2-Pad10)
- U1 pad 11: Net-(U1-PA3) -> unconnected-(U1-PA3-Pad11)
- U1 pad 12: DISCHARGE3 -> unconnected-(U1-PA4-Pad12)
- U1 pad 13: DISCHARGE2 -> DISCHARGE0
- U1 pad 14: DISCHARGE1 -> unconnected-(U1-PA6-Pad14)
- U1 pad 15: DISCHARGE0 -> ADC0
- U1 pad 25: unconnected-(U1-PB11-Pad25) -> DISCHARGE1
- U1 pad 26: Net-(U1-PB12) -> ADC1
- U1 pad 27: Net-(U1-PB13) -> DISCHARGE2
- U1 pad 28: Net-(U1-PB14) -> ADC2
- U1 pad 29: Net-(U1-PB15) -> unconnected-(U1-PB15-Pad29)
- U1 pad 8: Net-(U1-PA0) -> DISCHARGE3
- U1 pad 9: Net-(U1-PA1) -> ADC3
- U4 pad 24: +3.3VA -> +3.3V
- U5 pad 24: +3.3VA -> +3.3V
- U6 pad 24: +3.3VA -> +3.3V
- U7 pad 24: +3.3VA -> +3.3V
Routing:
- net D+: track 0.00 -> 85.6 mm
- net D-: track 0.00 -> 84.9 mm
- net SENSE2: track 154.9 -> 216.9 mm, vias 0 -> 1
- net +3.3V: track 0.00 -> 56.4 mm, vias 0 -> 6
- net +5V: track 0.00 -> 52.2 mm
- net SENSE0: track 141.3 -> 180.7 mm, vias 0 -> 1
- net SENSE1: track 218.9 -> 254.6 mm, vias 0 -> 1
- net +3.3VA: track 1.90 -> 26.7 mm, vias 1 -> 5
- net SENSE3: track 223.8 -> 244.5 mm, vias 0 -> 1
- net DISCHARGE2: track 0.00 -> 19.7 mm
- net +5V_USB: track 0.00 -> 19.4 mm, vias 0 -> 6
- net ADC2: track 0.00 -> 18.5 mm
- net ADC1: track 4.65 -> 20.4 mm
- net DISCHARGE1: track 4.72 -> 19.7 mm
- net DISCHARGE0: track 0.00 -> 10.3 mm
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
Commit message: 29.04.2026
Parts:
- moved J4 75.7 mm to (196.1, 88.5)
- moved C13 25.4 mm to (149.6, 94.1), turned to 0 degrees
- moved C17 22.4 mm to (160.3, 32.5), turned to 90 degrees
- moved U3 21.3 mm to (157.2, 32.5), turned to 0 degrees
- moved C16 20.6 mm to (154.4, 32.5), turned to 90 degrees
- moved C10 10.7 mm to (93.7, 33.3)
- moved C11 10.5 mm to (155.2, 52.0), turned to 90 degrees
- moved BOOT_SW1 9.25 mm to (188.5, 69.7)
- moved RESET_SW1 9.25 mm to (192.1, 69.7)
- moved C8 4.90 mm to (161.7, 76.1), turned to 0 degrees
- moved J5 3.70 mm to (148.4, 30.5)
- moved R31 2.93 mm to (165.1, 73.6)
- moved C12 2.54 mm to (207.2, 45.6), turned to -90 degrees
- moved C6 2.14 mm to (163.9, 76.2), turned to 90 degrees
- moved C9 2.02 mm to (80.6, 73.4)
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Connections:
- J4 pad 1: +5V -> RESET
- J4 pad 2: +3.3V -> SWDIO
- J4 pad 3: unconnected-(J4-Pin_3-Pad3) -> SWCLK
- J4 pad 4: GND -> SWO
- J4 pad 5: SWO -> GND
- J4 pad 6: SWCLK -> unconnected-(J4-Pin_6-Pad6)
- J4 pad 7: SWDIO -> unconnected-(J4-Pin_7-Pad7)
- J4 pad 8: RESET -> +3.3V
- SW1 pad 2: unconnected-(SW1-Pad2) -> MUX1_D3
- SW10 pad 2: unconnected-(SW10-Pad2) -> MUX3_D9
- SW11 pad 2: unconnected-(SW11-Pad2) -> MUX3_D10
- SW12 pad 2: unconnected-(SW12-Pad2) -> MUX3_D6
- SW13 pad 2: unconnected-(SW13-Pad2) -> MUX1_D4
- SW14 pad 2: unconnected-(SW14-Pad2) -> MUX1_D5
- SW15 pad 2: unconnected-(SW15-Pad2) -> MUX1_D6
- SW16 pad 2: unconnected-(SW16-Pad2) -> MUX1_D7
- SW17 pad 2: unconnected-(SW17-Pad2) -> MUX1_D14
- SW2 pad 2: unconnected-(SW2-Pad2) -> MUX1_D2
- SW22 pad 2: unconnected-(SW22-Pad2) -> MUX3_D8
- SW23 pad 2: unconnected-(SW23-Pad2) -> MUX3_D7
- SW24 pad 2: unconnected-(SW24-Pad2) -> MUX0_D12
- SW25 pad 2: unconnected-(SW25-Pad2) -> MUX0_D11
- SW26 pad 2: unconnected-(SW26-Pad2) -> MUX0_D10
- SW27 pad 2: unconnected-(SW27-Pad2) -> MUX0_D9
- SW28 pad 2: unconnected-(SW28-Pad2) -> MUX1_D13
- SW29 pad 2: unconnected-(SW29-Pad2) -> MUX2_D6
- SW3 pad 2: unconnected-(SW3-Pad2) -> MUX1_D1
- SW30 pad 2: unconnected-(SW30-Pad2) -> MUX2_D7
- SW32 pad 2: unconnected-(SW32-Pad2) -> MUX3_D11
- SW35 pad 2: unconnected-(SW35-Pad2) -> MUX0_D13
- SW36 pad 2: unconnected-(SW36-Pad2) -> MUX0_D14
- SW38 pad 2: unconnected-(SW38-Pad2) -> MUX0_D5
- SW39 pad 2: unconnected-(SW39-Pad2) -> MUX0_D7
- SW4 pad 2: unconnected-(SW4-Pad2) -> MUX1_D0
- SW40 pad 2: unconnected-(SW40-Pad2) -> MUX3_D12
- SW42 pad 2: unconnected-(SW42-Pad2) -> MUX3_D14
- SW43 pad 2: unconnected-(SW43-Pad2) -> MUX3_D15
- SW44 pad 2: unconnected-(SW44-Pad2) -> MUX3_D0
- SW45 pad 2: unconnected-(SW45-Pad2) -> MUX0_D15
- SW47 pad 2: unconnected-(SW47-Pad2) -> MUX3_D13
- SW49 pad 2: unconnected-(SW49-Pad2) -> MUX0_D6
- SW5 pad 2: unconnected-(SW5-Pad2) -> MUX1_D15
Routing:
- net +3.3V: track 56.4 -> 282.0 mm, vias 6 -> 10
- net MUX0_D12: track 0.00 -> 76.6 mm
- net MUX0_D7: track 0.00 -> 71.5 mm
- net MUX1_D3: track 0.00 -> 68.9 mm
- net MUX0_D13: track 0.00 -> 59.8 mm
- net MUX1_D4: track 0.00 -> 57.6 mm
- net MUX3_D14: track 0.00 -> 55.2 mm
- net MUX0_D11: track 0.00 -> 51.8 mm
- net MUX1_D2: track 0.00 -> 49.8 mm
- net MUX3_D9: track 0.00 -> 48.6 mm
- net MUX0_D6: track 0.00 -> 47.2 mm
- net MUX0_D14: track 0.00 -> 38.4 mm
- net MUX1_D13: track 0.00 -> 37.0 mm
- net MUX3_D8: track 0.00 -> 36.1 mm
- net MUX1_D5: track 0.00 -> 35.9 mm
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
Commit message: 30.04.2026
Parts:
- removed the C13 at (149.6, 94.1)
- removed the R11 at (119.2, 108.6)
- removed the R12 at (119.2, 111.1)
- removed R25, R26, R27, R28, R31, R32: 330, Resistor_SMD:R_0603_1608Metric
- removed the R37 at (115.2, 113.6)
- removed the R38 at (115.2, 116.1)
- removed the R5 at (119.2, 103.6)
- removed the R6 at (119.2, 106.1)
- SW18, SW19, SW20, SW21: footprint Kicad footprints:ecs_pad_1U_hybrid_hotswap_V3 -> Kicad footprints:ecs_pad_1U_hybrid_hotswap_V3_switched_sides
- moved U4 57.4 mm to (35.3, 48.0), turned to 0 degrees
- moved C9 46.0 mm to (40.1, 51.6), turned to 0 degrees
- moved R12 39.5 mm to (156.8, 95.2)
- moved U5 19.6 mm to (93.7, 48.8)
- moved C10 19.6 mm to (98.5, 52.4)
- moved R83 16.0 mm to (165.5, 78.6), turned to 0 degrees
- moved C19 14.6 mm to (174.6, 92.5)
- moved C23 14.6 mm to (177.8, 97.2)
- moved R90 14.6 mm to (174.6, 97.2)
- moved U9 14.6 mm to (176.6, 94.5)
- moved R82 14.6 mm to (180.9, 97.2)
- moved R86 14.6 mm to (173.8, 94.5)
- moved R91 10.8 mm to (156.0, 77.8)
- moved C20 10.8 mm to (158.4, 75.8)
- moved R87 10.8 mm to (157.6, 77.8)
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- renumbered C14 to C13, C15 to C14, C16 to C15, C17 to C16, J5 to J4, J4 to J5, R31 to R11, R32 to R12, R19 to R5, R20 to R6
Connections:
- J5 pad 1: RESET -> BOOT0
- J5 pad 2: SWDIO -> SWO
- J5 pad 4: SWO -> SWDIO
- J5 pad 6: unconnected-(J4-Pin_6-Pad6) -> RESET
- SW16 pad 2: MUX1_D7 -> MUX1_D8
- SW18 pad 2: unconnected-(SW18-Pad2) -> MUX2_D3
- SW19 pad 2: unconnected-(SW19-Pad2) -> MUX2_D2
- SW20 pad 2: unconnected-(SW20-Pad2) -> MUX2_D8
- SW21 pad 2: unconnected-(SW21-Pad2) -> MUX2_D13
- SW31 pad 2: unconnected-(SW31-Pad2) -> MUX2_D10
- SW5 pad 2: MUX1_D15 -> MUX1_D7
- SW6 pad 2: unconnected-(SW6-Pad2) -> MUX2_D5
- SW7 pad 2: unconnected-(SW7-Pad2) -> MUX2_D4
- SW8 pad 2: unconnected-(SW8-Pad2) -> MUX2_D12
- SW9 pad 2: unconnected-(SW9-Pad2) -> MUX2_D11
- U1 pad 10: unconnected-(U1-PA2-Pad10) -> MUX1_IN
- U1 pad 11: unconnected-(U1-PA3-Pad11) -> MUX0_IN
- U1 pad 31: unconnected-(U1-PA9-Pad31) -> MUX3_IN
- U1 pad 32: unconnected-(U1-PA10-Pad32) -> MUX2_IN
Routing:
- net +3.3V: track 282.0 -> 0.00 mm, vias 10 -> 0
- net SENSE3: track 257.9 -> 0.00 mm, vias 1 -> 0
- net SENSE1: track 240.4 -> 0.00 mm, vias 1 -> 0
- net SENSE2: track 224.8 -> 0.00 mm, vias 1 -> 0
- net SENSE0: track 180.7 -> 0.00 mm, vias 1 -> 0
- net D+: track 83.5 -> 0.00 mm
- net D-: track 82.9 -> 0.00 mm
- net MUX0_D12: track 76.6 -> 0.00 mm
- net MUX0_D7: track 71.5 -> 0.00 mm
- net MUX1_D3: track 68.9 -> 0.00 mm
- net MUX0_D13: track 59.8 -> 0.00 mm
- net MUX1_D4: track 57.6 -> 0.00 mm
- net MUX3_D14: track 55.2 -> 0.00 mm
- net MUX0_D11: track 51.8 -> 0.00 mm
- net MUX1_D2: track 49.8 -> 0.00 mm
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Other:
- board text added: "Daisy40 inspired hybrid pcb by FriedSoul STM32-2L v0.9 2026"
- board text added: "TOPREN'T"

Commit message: 14.05.2026
Parts:
- added C17: 15pF, Capacitor_SMD:C_0402_1005Metric, B.Cu at (167.5, 86.9)
- added C26: 15pF, Capacitor_SMD:C_0402_1005Metric, B.Cu at (164.3, 86.5)
- added Y1: Crystal_GND24_Small, Crystal:Crystal_SMD_3225-4Pin_3.2x2.5mm, B.Cu at (166.3, 84.5)
- moved C15 56.8 mm to (209.9, 33.3), turned to 180 degrees
- moved U3 54.1 mm to (209.9, 36.1), turned to -90 degrees
- moved C16 51.2 mm to (209.9, 39.3), turned to 180 degrees
- moved R90 50.7 mm to (124.2, 103.2), turned to 90 degrees
- moved R92 48.9 mm to (140.5, 102.8)
- moved C19 48.8 mm to (126.6, 101.2)
- moved U9 48.8 mm to (128.6, 103.2)
- moved R86 48.8 mm to (125.8, 103.2)
- moved R82 47.7 mm to (133.7, 104.0)
- moved C23 46.8 mm to (131.4, 103.2), turned to 90 degrees
- moved R89 46.4 mm to (142.1, 102.8), turned to 90 degrees
- moved C21 44.4 mm to (142.9, 100.8), turned to 0 degrees
- moved R84 44.1 mm to (150.0, 103.6), turned to 0 degrees
- moved U11 42.7 mm to (144.9, 102.8), turned to 180 degrees
- moved C25 40.6 mm to (147.6, 102.8), turned to 90 degrees
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Connections:
- J5 pad 6: RESET -> unconnected-(J5-Pin_6-Pad6)
- J5 pad 7: unconnected-(J5-Pin_7-Pad7) -> +3.3V
- J5 pad 8: +3.3V -> RESET
- U1 pad 5: unconnected-(U1-PF0-Pad5) -> Net-(U1-PF0)
- U1 pad 6: unconnected-(U1-PF1-Pad6) -> Net-(U1-PF1)
Routing:
- net +3.3V: track 0.00 -> 236.6 mm, vias 0 -> 9
- net D+: track 0.00 -> 70.1 mm
- net D-: track 0.00 -> 69.0 mm
- net RESET: track 0.00 -> 20.3 mm, vias 0 -> 2
- net +5V_USB: track 0.00 -> 19.4 mm, vias 0 -> 6
- net SWDIO: track 0.00 -> 10.5 mm
- net SWCLK: track 0.00 -> 9.72 mm
- net SWO: track 0.00 -> 8.78 mm
- net BOOT0: track 0.00 -> 7.78 mm, vias 0 -> 1
- net Net-(U1-PF1): track 0.00 -> 7.17 mm
- net Net-(U1-PF0): track 0.00 -> 5.59 mm
- net +5V: track 0.00 -> 5.31 mm
- net GND: track 0.00 -> 2.90 mm

Commit message: 15.05.2026
Parts:
- moved BOOT_SW1 104.5 mm to (88.1, 79.4)
- moved RESET_SW1 104.5 mm to (84.5, 79.4)
- moved R81 59.9 mm to (79.4, 77.0), turned to -90 degrees
- moved C22 58.4 mm to (79.8, 73.4)
- moved U8 58.1 mm to (77.0, 74.2), turned to -90 degrees
- moved C18 56.6 mm to (75.0, 76.2), turned to 90 degrees
- moved R85 54.5 mm to (77.0, 77.0), turned to 180 degrees
- moved R88 52.4 mm to (77.0, 78.6), turned to 180 degrees
- moved R92 51.6 mm to (177.8, 67.1)
- moved C15 49.3 mm to (160.7, 31.4), turned to 90 degrees
- moved R89 48.0 mm to (177.0, 69.9), turned to -45 degrees
- moved U3 46.7 mm to (163.5, 31.4), turned to 0 degrees
- moved C21 45.4 mm to (177.8, 71.8), turned to -135 degrees
- moved C16 44.0 mm to (166.7, 31.4), turned to 90 degrees
- moved R84 43.4 mm to (175.2, 68.3), turned to -135 degrees
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Routing:
- net +3.3V: track 236.6 -> 84.7 mm
- net +5V_USB: track 19.4 -> 161.1 mm, vias 6 -> 4
- net DM_USB: track 0.00 -> 43.6 mm
- net DP_USB: track 0.00 -> 42.9 mm
- net +5V: track 5.31 -> 30.5 mm
- net D-: track 69.0 -> 83.6 mm
- net D+: track 70.1 -> 84.4 mm
- net RESET: track 20.3 -> 10.3 mm, vias 2 -> 1
- net SWDIO: track 10.5 -> 2.03 mm
- net SWCLK: track 9.72 -> 2.03 mm
- net SWO: track 8.78 -> 2.03 mm
- net BOOT0: track 7.78 -> 2.03 mm, vias 1 -> 0
- net Net-(J2-CC1): track 0.00 -> 2.08 mm
- net Net-(J3-CC1): track 0.00 -> 2.08 mm
- net Net-(J1-CC1): track 0.00 -> 2.08 mm
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