File: Romashka EC non-matrix/Romashka EC non-matrix.kicad_pcb (KiCad board)
At the start: 2 copper layers, 228.6 x 76.2 mm, 167 parts, among them J1 Daisy40, J2 RS40, J3 JJ40, J4 JSB USB, J5 SOICbite, SW1 EC_SW, SW10 EC_SW, SW11 EC_SW, SW12 EC_SW, SW13 EC_SW, SW14 EC_SW, SW15 EC_SW, SW16 EC_SW, SW17 EC_SW, SW18 EC_SW, SW19 EC_SW, SW2 EC_SW, SW20 EC_SW, SW21 EC_SW, SW22 EC_SW, SW23 EC_SW, SW24 EC_SW, SW25 EC_SW, SW26 EC_SW, SW27 EC_SW, SW28 EC_SW, SW29 EC_SW, SW3 EC_SW, SW30 EC_SW, SW31 EC_SW, SW32 EC_SW, SW35 EC_SW, SW36 EC_SW, SW38 EC_SW, SW39 EC_SW, SW4 EC_SW, SW40 EC_SW, SW42 EC_SW, SW43 EC_SW, SW44 EC_SW, SW45 EC_SW, SW47 EC_SW, SW49 EC_SW, SW5 EC_SW, SW6 EC_SW, SW7 EC_SW, SW8 EC_SW, SW9 EC_SW, U1 STM32G474CBTx, U10 TLV9061xDBV, U11 TLV9061xDBV, U2 USBLC6-2P6, U3 TPS7A2033, U4 HEF4067BTT, U5 HEF4067BTT, U6 HEF4067BTT, U7 HEF4067BTT, U8 TLV9061xDBV, U9 TLV9061xDBV, Y1 Crystal_GND24_Small

Commit message: 25.05.2026
Parts:
- moved C22 0.89 mm to (65.6, 69.3)
- moved R88 0.89 mm to (60.7, 66.7)
- moved R85 0.89 mm to (62.3, 66.7)
- moved U8 0.89 mm to (65.1, 66.7)
- moved C18 0.89 mm to (63.1, 64.7)
- moved R81 0.89 mm to (62.5, 69.1)
Connections:
- C18 pad 2: +3.3VA -> +3.3V
- C19 pad 2: +3.3VA -> +3.3V
- C20 pad 2: +3.3VA -> +3.3V
- C21 pad 2: +3.3VA -> +3.3V
- U10 pad 5: +3.3VA -> +3.3V
- U11 pad 5: +3.3VA -> +3.3V
- U8 pad 5: +3.3VA -> +3.3V
- U9 pad 5: +3.3VA -> +3.3V
Routing:
- net +3.3V: track 307.6 -> 360.3 mm, vias 11 -> 17
- net MUX0_IN: track 168.9 -> 132.9 mm
- net SENSE1: track 214.9 -> 198.8 mm
- net +3.3VA: track 10.5 -> 0.00 mm, vias 4 -> 0
- net SENSE0: track 269.9 -> 277.7 mm, vias 0 -> 1
- net MUX_S3: track 234.7 -> 234.0 mm
- net SENSE2: track 189.0 -> 188.5 mm
- net GND: vias 16 -> 13

Commit message: 25.05.2026
Parts:
- SW24, SW25: footprint Kicad footprints:ecs_pad_1U_hybrid_hotswap_V3 -> Kicad footprints:ecs_pad_1U_hybrid_hotswap_V3_switched_sides
- moved R88 8.87 mm to (64.7, 58.7)
- moved R81 7.79 mm to (63.1, 61.3), turned to 90 degrees
- moved R85 6.40 mm to (65.5, 61.1), turned to 0 degrees
- moved C22 5.56 mm to (62.9, 64.4), turned to -90 degrees
- moved C18 5.17 mm to (67.5, 61.9), turned to -90 degrees
- moved U8 2.81 mm to (65.5, 63.9), turned to 90 degrees
- moved R92 2.14 mm to (141.7, 59.9), turned to 0 degrees
- moved C21 1.19 mm to (143.7, 62.3)
- moved U11 1.19 mm to (141.7, 64.3)
- moved C25 1.19 mm to (139.2, 64.8)
- moved R84 1.19 mm to (139.4, 61.7)
- moved R89 1.19 mm to (141.7, 61.5)
- moved C20 0.79 mm to (124.6, 61.9)
- moved C24 0.79 mm to (120.1, 64.4)
- moved R83 0.79 mm to (120.3, 61.3)
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Routing:
- net MUX1_D7: track 33.5 -> 0.01 mm
- net MUX0_D7: track 23.7 -> 0.00 mm
- net MUX1_D6: track 15.0 -> 0.00 mm
- net MUX1_D2: track 12.5 -> 0.00 mm
- net MUX0_D1: track 5.22 -> 17.6 mm
- net MUX0_IN: track 132.9 -> 143.5 mm
- net SENSE0: track 277.7 -> 267.3 mm, vias 1 -> 0
- net +3.3V: track 360.3 -> 368.8 mm
- net MUX_S1: track 222.6 -> 217.9 mm, vias 9 -> 8
- net MUX_S0: track 227.8 -> 223.5 mm, vias 9 -> 8
- net MUX_S2: track 234.3 -> 230.4 mm, vias 9 -> 8
- net MUX_S3: track 234.0 -> 230.8 mm, vias 9 -> 8
- net SENSE1: track 198.8 -> 195.9 mm
- net MUX1_IN: track 106.7 -> 107.7 mm
- net MUX1_D1: track 36.7 -> 37.7 mm
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
Commit message: 26.05.2026
Parts:
- SW32: footprint Kicad footprints:ecs_pad_1U_hybrid_hotswap_V3 -> Kicad footprints:ecs_pad_1U_hybrid_hotswap_V3_switched_sides
- moved R84 59.5 mm to (170.4, 112.4), turned to 0 degrees
- moved C25 58.9 mm to (173.6, 112.6), turned to 0 degrees
- moved R89 56.4 mm to (170.3, 110.1), turned to 90 degrees
- moved U11 55.5 mm to (173.1, 110.1), turned to 180 degrees
- moved R92 55.0 mm to (170.3, 106.9), turned to 90 degrees
- moved C21 53.7 mm to (172.3, 107.7), turned to 180 degrees
- moved R83 19.1 mm to (139.4, 61.3)
- moved R91 19.0 mm to (140.9, 58.7)
- moved C20 19.0 mm to (143.7, 61.9)
- moved C24 19.0 mm to (139.2, 64.4)
- moved R87 19.0 mm to (141.7, 61.1)
- moved U10 19.0 mm to (141.7, 63.9)
- moved C12 10.8 mm to (206.8, 50.4), turned to 90 degrees
- moved C10 10.5 mm to (88.9, 51.6), turned to -90 degrees
- moved C11 10.5 mm to (146.1, 51.6), turned to -90 degrees
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Routing:
- net MUX_S3: track 230.8 -> 95.9 mm, vias 8 -> 1
- net MUX_S2: track 230.4 -> 101.4 mm, vias 8 -> 2
- net MUX_S0: track 223.5 -> 104.3 mm, vias 8 -> 4
- net MUX_S1: track 217.9 -> 99.5 mm, vias 8 -> 1
- net +3.3V: track 368.8 -> 267.0 mm, vias 17 -> 14
- net MUX0_IN: track 143.5 -> 65.7 mm, vias 4 -> 2
- net MUX3_IN: track 60.6 -> 4.91 mm, vias 2 -> 0
- net MUX1_IN: track 107.7 -> 53.5 mm, vias 4 -> 1
- net MUX2_IN: track 52.4 -> 5.69 mm, vias 2 -> 0
- net MUX3_D6: track 35.7 -> 0.00 mm
- net MUX1_D0: track 29.9 -> 0.00 mm
- net MUX0_D15: track 26.8 -> 0.00 mm
- net MUX3_D7: track 21.2 -> 0.50 mm
- net MUX3_D0: track 17.3 -> 0.00 mm
- net MUX2_D10: track 30.4 -> 18.5 mm
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
Commit message: 26.05.2026
Parts:
- moved R84 52.7 mm to (158.4, 61.1), turned to -90 degrees
- moved C25 50.8 mm to (158.0, 64.3), turned to -90 degrees
- moved R89 49.9 mm to (160.7, 61.1), turned to 0 degrees
- moved R92 49.3 mm to (159.9, 58.7)
- moved U11 47.8 mm to (160.7, 63.9), turned to 90 degrees
- moved C21 46.8 mm to (162.7, 61.9), turned to -90 degrees
Routing:
- net Net-(U11--): track 5.40 -> 0.00 mm
- net ADC2: track 4.65 -> 0.00 mm
- net DISCHARGE2: track 4.25 -> 0.00 mm
- net +3.3V: track 267.0 -> 264.7 mm, vias 14 -> 13
