File: Romashka EC non-matrix/Romashka EC non-matrix.kicad_pcb (KiCad board)
At the start: 2 copper layers, 228.6 x 76.2 mm, 167 parts, among them J1 Daisy40, J2 RS40, J3 JJ40, J4 JSB USB, J5 SOICbite, SW1 EC_SW, SW10 EC_SW, SW11 EC_SW, SW12 EC_SW, SW13 EC_SW, SW14 EC_SW, SW15 EC_SW, SW16 EC_SW, SW17 EC_SW, SW18 EC_SW, SW19 EC_SW, SW2 EC_SW, SW20 EC_SW, SW21 EC_SW, SW22 EC_SW, SW23 EC_SW, SW24 EC_SW, SW25 EC_SW, SW26 EC_SW, SW27 EC_SW, SW28 EC_SW, SW29 EC_SW, SW3 EC_SW, SW30 EC_SW, SW31 EC_SW, SW32 EC_SW, SW35 EC_SW, SW36 EC_SW, SW38 EC_SW, SW39 EC_SW, SW4 EC_SW, SW40 EC_SW, SW42 EC_SW, SW43 EC_SW, SW44 EC_SW, SW45 EC_SW, SW47 EC_SW, SW49 EC_SW, SW5 EC_SW, SW6 EC_SW, SW7 EC_SW, SW8 EC_SW, SW9 EC_SW, U1 STM32G474CBTx, U10 TLV9061xDBV, U11 TLV9061xDBV, U2 USBLC6-2P6, U3 TPS7A2033, U4 HEF4067BTT, U5 HEF4067BTT, U6 HEF4067BTT, U7 HEF4067BTT, U8 TLV9061xDBV, U9 TLV9061xDBV, Y1 Crystal_GND24_Small

Commit message: 07.07.2026
Parts:
- moved F1 7.55 mm to (135.3, 31.8)
Routing:
- net MUX0_IN: track 65.7 -> 110.4 mm, vias 2 -> 3
- net MUX_S3: track 95.9 -> 124.3 mm
- net MUX_S1: track 99.5 -> 126.3 mm
- net SENSE1: track 197.2 -> 178.5 mm
- net MUX2_D10: track 18.5 -> 9.91 mm
- net +5V_USB: track 45.5 -> 37.7 mm
- net SENSE2: track 188.2 -> 193.6 mm
- net MUX_S0: track 104.3 -> 99.1 mm, vias 4 -> 5
- net +5V: track 32.5 -> 34.6 mm
- net MUX_S2: track 101.4 -> 99.4 mm, vias 2 -> 3
- net SENSE3: track 257.9 -> 256.0 mm
- net SENSE0: track 267.3 -> 265.5 mm
- net MUX1_IN: track 53.5 -> 52.2 mm

Commit message: 20.08.2026
Parts:
- SW1, SW2, SW3, SW35, SW40, SW42, SW6, SW7: footprint Kicad footprints:ecs_pad_1U_hybrid_hotswap_V3 -> FriedSoul_switches:ecs_pad_1U_hybrid_hotswap_V3
- SW10, SW11, SW12, SW13, SW14, SW15, SW16, SW17, SW18, SW19, SW20, SW21, SW22, SW23, SW24, SW25, SW26, SW27, SW28, SW29, SW30, SW31, SW32, SW38, SW39, SW4, SW5, SW8, SW9: footprint Kicad footprints:ecs_pad_1U_hybrid_hotswap_V3_switched_sides -> FriedSoul_switches:ecs_pad_1U_hybrid_hotswap_V3_switched_sides
- SW36, SW43, SW44, SW45, SW47: footprint Kicad footprints:ecs_pad_hybrid_hotswap_2.381_V3 -> FriedSoul_switches:ecs_pad_hybrid_hotswap_2.381_V3
- SW49: footprint Kicad footprints:ecs_pad_hybrid_hotswap_7.144_V3 -> FriedSoul_switches:ecs_pad_hybrid_hotswap_7.144_V3
- moved F1 7.55 mm to (142.9, 32.1)
Routing:
- net MUX0_IN: track 110.4 -> 65.7 mm, vias 3 -> 2
- net MUX_S3: track 124.3 -> 95.9 mm
- net MUX_S1: track 126.3 -> 99.5 mm
- net SENSE1: track 178.5 -> 197.2 mm
- net MUX2_D10: track 9.91 -> 18.5 mm
- net +5V_USB: track 37.7 -> 45.5 mm
- net SENSE2: track 193.6 -> 188.2 mm
- net MUX_S0: track 99.1 -> 104.3 mm, vias 5 -> 4
- net +5V: track 34.6 -> 32.5 mm
- net MUX_S2: track 99.4 -> 101.4 mm, vias 3 -> 2
- net SENSE3: track 256.0 -> 257.9 mm
- net SENSE0: track 265.5 -> 267.3 mm
- net MUX1_IN: track 52.2 -> 53.5 mm

Commit message: 20.08.2026
Parts:
- removed C13: 10uF, Capacitor_SMD:C_0805_2012Metric
- removed R59, R74: 100K, Resistor_SMD:R_0603_1608Metric
- moved C11 19.1 mm to (127.0, 50.8), turned to 90 degrees
- moved U6 19.1 mm to (131.8, 48.0)
- moved F1 8.34 mm to (134.5, 31.8)
- moved C10 0.79 mm to (88.9, 50.8), turned to 90 degrees
Connections:
- U1 pad 32: unconnected-(U1-PA10-Pad32) -> MUX_EN
- U4 pad 15: GND -> MUX_EN
- U5 pad 15: GND -> MUX_EN
- U6 pad 15: GND -> MUX_EN
- U7 pad 15: GND -> MUX_EN
Routing:
- net ADC0: track 4.65 -> 110.2 mm, vias 0 -> 1
- net MUX_S0: track 104.3 -> 1.14 mm, vias 4 -> 1
- net DISCHARGE0: track 4.31 -> 105.6 mm, vias 0 -> 1
- net MUX_S2: track 101.4 -> 1.14 mm, vias 2 -> 1
- net MUX_S1: track 99.5 -> 1.14 mm
- net MUX_S3: track 95.9 -> 2.15 mm
- net MUX0_IN: track 65.7 -> 0.00 mm, vias 2 -> 0
- net +3.3V: track 264.7 -> 201.7 mm, vias 13 -> 12
- net MUX1_IN: track 53.5 -> 0.00 mm, vias 1 -> 0
- net MUX2_D6: track 0.00 -> 36.4 mm
- net SENSE2: track 188.2 -> 165.9 mm
- net MUX2_D2: track 0.00 -> 22.0 mm
- net +5V_USB: track 45.5 -> 36.9 mm
- net MUX2_IN: track 5.69 -> 0.00 mm
- net MUX3_IN: track 4.91 -> 0.00 mm
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
Commit message: 21.08.2026
Parts:
- SW35: footprint FriedSoul_switches:ecs_pad_1U_hybrid_hotswap_V3 -> FriedSoul_switches:ecs_pad_1U_hybrid_hotswap_V3_switched_sides
- SW39: footprint FriedSoul_switches:ecs_pad_1U_hybrid_hotswap_V3_switched_sides -> FriedSoul_switches:ecs_pad_1U_hybrid_hotswap_V3
- moved BOOT_SW1 85.0 mm to (172.6, 92.9)
- moved RESET_SW1 85.0 mm to (169.1, 92.9)
- moved C22 60.1 mm to (122.8, 69.3), turned to 45 degrees
- moved R81 58.2 mm to (120.5, 71.4), turned to -135 degrees
- moved U8 55.3 mm to (120.7, 67.9), turned to -135 degrees
- moved R88 54.3 mm to (117.6, 71.0), turned to 135 degrees
- moved R85 53.9 mm to (118.7, 69.8), turned to 135 degrees
- moved C18 50.7 mm to (117.8, 67.9), turned to 45 degrees
- moved R92 23.3 mm to (156.4, 81.8), turned to 180 degrees
- moved R84 22.2 mm to (158.9, 83.3), turned to 0 degrees
- moved R89 19.9 mm to (158.8, 81.0), turned to 90 degrees
- moved C25 19.6 mm to (162.1, 83.5), turned to 0 degrees
- moved C11 19.1 mm to (146.1, 50.8)
- moved U6 19.1 mm to (150.8, 48.0)
- moved C21 17.4 mm to (159.5, 79.0), turned to 0 degrees
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Connections:
- J5 pad 6: +3.3V -> GND
- J5 pad 7: GND -> +3.3V
- SW15 pad 1: SENSE0 -> SENSE1
- SW38 pad 1: SENSE1 -> SENSE0
- U1 pad 10: unconnected-(U1-PA2-Pad10) -> DISCHARGE1
- U1 pad 11: unconnected-(U1-PA3-Pad11) -> ADC1
- U1 pad 30: unconnected-(U1-PA8-Pad30) -> ADC3
- U1 pad 44: unconnected-(U1-PB7-Pad44) -> DISCHARGE2
- U1 pad 8: unconnected-(U1-PA0-Pad8) -> DISCHARGE3
- U1 pad 9: DISCHARGE2 -> unconnected-(U1-PA1-Pad9)
Routing:
- net ADC0: track 110.2 -> 4.65 mm, vias 1 -> 0
- net DISCHARGE0: track 105.6 -> 4.31 mm, vias 1 -> 0
- net +3.3V: track 201.7 -> 120.0 mm
- net MUX0_D6: track 38.2 -> 0.13 mm
- net MUX2_D6: track 36.4 -> 0.00 mm
- net MUX0_D11: track 35.5 -> 0.00 mm
- net MUX1_D11: track 35.4 -> 0.00 mm
- net MUX0_D0: track 27.5 -> 0.00 mm
- net MUX1_D1: track 26.8 -> 0.00 mm
- net MUX0_D2: track 25.8 -> 0.00 mm
- net MUX1_D7: track 0.01 -> 23.6 mm
- net MUX2_D2: track 22.0 -> 0.00 mm
- net SENSE1: track 195.7 -> 208.3 mm
- net MUX0_D7: track 0.00 -> 9.44 mm
- net MUX2_D7: track 0.00 -> 7.19 mm
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