File: Romashka EC non-matrix/Logic.kicad_sch (KiCad schematic)
At the start: 107 parts, among them SW1 EC_SW, SW10 EC_SW, SW11 EC_SW, SW12 EC_SW, SW13 EC_SW, SW14 EC_SW, SW15 EC_SW, SW16 EC_SW, SW17 EC_SW, SW18 EC_SW, SW19 EC_SW, SW2 EC_SW, SW20 EC_SW, SW21 EC_SW, SW22 EC_SW, SW23 EC_SW, SW24 EC_SW, SW25 EC_SW, SW26 EC_SW, SW27 EC_SW, SW28 EC_SW, SW29 EC_SW, SW3 EC_SW, SW30 EC_SW, SW31 EC_SW, SW32 EC_SW, SW33 EC_SW, SW34 EC_SW, SW35 EC_SW, SW36 EC_SW, SW37 EC_SW, SW38 EC_SW, SW39 EC_SW, SW4 EC_SW, SW40 EC_SW, SW41 EC_SW, SW42 EC_SW, SW43 EC_SW, SW44 EC_SW, SW45 EC_SW, SW46 EC_SW, SW47 EC_SW, SW48 EC_SW, SW49 EC_SW, SW5 EC_SW, SW6 EC_SW, SW7 EC_SW, SW8 EC_SW, SW9 EC_SW, U10 TLV9061xDBV, U11 TLV9061xDBV, U12 TLV9061xDBV, U13 TLV9061xDBV, U14 TLV9061xDBV, U15 TLV9061xDBV, U4 4051, U5 4051, U6 4051, U7 4051, U8 4051, U9 4051

Commit message: 24.04.2026
Parts:
- removed C13, C14, C36, C37: 100nF, Capacitor_SMD:C_0402_1005Metric, symbol Device:C_Small
- removed C22, C24, C26, C28, C30, C32: 1uF, Capacitor_SMD:C_0603_1608Metric, symbol Device:C_Small
- removed C29, C31: 470pF, Capacitor_SMD:C_0603_1608Metric, symbol Device:C_Small
- removed R19: 33K, Resistor_SMD:R_0603_1608Metric, symbol Device:R_Small
- removed R20, R25, R26: 330, Resistor_SMD:R_0603_1608Metric, symbol Device:R_Small
- removed U14, U15: TLV9061xDBV, Package_TO_SOT_SMD:SOT-23-5, symbol Amplifier_Operational:TLV9061xDBV
- removed U4, U5, U6, U7, U8, U9: 4051, Package_SO:Texas_DYY0016A_TSOT-23-16_2x4.2mm_P0.5mm, symbol 4xxx:4051
- added R10, R13, R14, R15, R16, R21, R22, R23, R24, R29, R30, R33, R34, R35, R36, R37, R38, R39, R40, R41, R42, R43, R44, R45, R46, R47, R48, R49, R50, R51, R52, R53, R54, R55, R56, R57, R58, R59, R60, R61, R62, R63, R64, R65, R66, R67, R68, R69, R7, R70, R71, R72, R73, R74, R75, R76, R77, R78, R79, R8, R80, R9: 100K, Resistor_SMD:R_0603_1608Metric, symbol Device:R_Small
- added U4, U5, U6, U7: HEF4067BTT, Package_SO:TSSOP-24_4.4x7.8mm_P0.65mm, symbol Analog_Switch:HEF4067BTT
- R17: value 33K -> 100K; now not fitted; now left out of the parts list
- R18: value 330 -> 100K; now not fitted; now left out of the parts list
- SW14, SW15, SW16, SW17, SW18, SW20, SW21, SW22, SW32: footprint Kicad footprints:ecs_pad_1U_hybrid_hotswap_V3_switched_sides -> Kicad footprints:ecs_pad_1U_hybrid_hotswap_V3
- SW23, SW24, SW29, SW39, SW40: footprint Kicad footprints:ecs_pad_1U_hybrid_hotswap_V3 -> Kicad footprints:ecs_pad_1U_hybrid_hotswap_V3_switched_sides
- renumbered C20 to C18, C35 to C19, C33 to C20, C34 to C21, C21 to C22, C27 to C23, C23 to C24, R21 to R81, R24 to R82, R22 to R83, R23 to R84, R7 to R85, R15 to R86, R9 to R87, R8 to R88, R13 to R89, R16 to R90, R10 to R91, R14 to R92, U11 to U10, U12 to U11, U10 to U8, U13 to U9
Connections:
- net ADC4 is gone; now on net MUX0_D4: R17.2
- net +3.3VA: now also U4.24 (VDD), U5.24 (VDD), U6.24 (VDD), U7.24 (VDD)
- net GND: now also R17.1, R18.1, R10.1, R13.1, R14.1, R15.1, R16.1, R21.1, R22.1, R23.1, R24.1, R29.1, R30.1, R33.1, R34.1, R35.1, R36.1, R37.1, R38.1, R39.1, R40.1, R41.2, R42.2, R43.2, R44.2, R45.2, R46.2, R47.2, R48.2, R49.2, R50.2, R51.2, R52.2, R53.2, R54.2, R55.2, R56.2, R57.2, R58.2, R59.2, R60.2, R61.2, R62.2, R63.2, R64.2, R65.2, R66.2, R67.2, R68.2, R69.2, R7.1, R70.2, R71.2, R72.2, R73.2, R74.2, R75.2, R76.2, R77.2, R78.2, R79.2, R8.1, R80.2, R9.1, U4.12 (VSS), U4.15 (~{E}), U5.12 (VSS), U5.15 (~{E}), U6.12 (VSS), U6.15 (~{E}), U7.12 (VSS), U7.15 (~{E}); no longer R18.2
- net MUX0_D0: now also R15.2, U4.9 (Y0); no longer SW49.2
- net MUX0_D1: now also R7.2, U4.8 (Y1); no longer SW38.2
- net MUX0_D2: now also R16.2, U4.7 (Y2); no longer SW45.2
- net MUX0_D3: now also R8.2, U4.6 (Y3); no longer SW39.2
- net MUX0_D4: now also U4.5 (Y4); no longer SW36.2
- net MUX0_D5: now also R9.2, U4.4 (Y5); no longer SW13.2
- net MUX0_D6: now also R55.1, U4.3 (Y6); no longer SW35.2
- net MUX0_D7: now also R45.1, U4.2 (Y7); no longer SW24.2
- net MUX0_IN: now also U4.1 (Z), U5.1 (Z), U6.1 (Z), U7.1 (Z)
- net MUX1_D0: now also R23.2, U5.9 (Y0)
- net MUX1_D1: now also R10.2, U5.8 (Y1)
- net MUX1_D2: now also R24.2, U5.7 (Y2)
- net MUX1_D3: now also R13.2, U5.6 (Y3)
- net MUX1_D4: now also R29.2, U5.5 (Y4)
- net MUX1_D5: now also R14.2, U5.4 (Y5)
- net MUX1_D6: now also R65.1, U5.3 (Y6)
- net MUX1_D7: now also R50.1, U5.2 (Y7)
- net MUX2_D0: now also R35.2, U6.9 (Y0)
- net MUX2_D1: now also R18.2, U6.8 (Y1)
- net MUX2_D2: now also R36.2, U6.7 (Y2)
- net MUX2_D3: now also R21.2, U6.6 (Y3)
- net MUX2_D4: now also R37.2, U6.5 (Y4)
- net MUX2_D5: now also R22.2, U6.4 (Y5)
- net MUX2_D6: now also R75.1, U6.3 (Y6)
- net MUX2_D7: now also R60.1, U6.2 (Y7)
- net MUX3_D0: now also R38.2, U7.9 (Y0)
- net MUX3_D1: now also R30.2, U7.8 (Y1)
- net MUX3_D2: now also R39.2, U7.7 (Y2)
- net MUX3_D3: now also R33.2, U7.6 (Y3)
- net MUX3_D4: now also R40.2, U7.5 (Y4)
- net MUX3_D5: now also R34.2, U7.4 (Y5)
- net MUX3_D6: now also R80.1, U7.3 (Y6)
- net MUX3_D7: now also R70.1, U7.2 (Y7)
- net MUX_S0: now also U4.10 (A0), U5.10 (A0), U6.10 (A0), U7.10 (A0)
- net MUX_S1: now also U4.11 (A1), U5.11 (A1), U6.11 (A1), U7.11 (A1)
- net MUX_S2: now also U4.14 (A2), U5.14 (A2), U6.14 (A2), U7.14 (A2)
- net SENSE0: now also SW10.1, SW11.1, SW12.1, SW2.1, SW23.1, SW3.1, SW4.1, SW5.1, SW6.1, SW7.1, SW8.1, SW9.1; no longer SW13.1, SW24.1, SW35.1, SW36.1, SW38.1, SW39.1, SW45.1, SW49.1
- net SENSE1: now also SW13.1, SW15.1, SW16.1, SW17.1, SW18.1, SW19.1, SW20.1, SW21.1, SW22.1; no longer SW2.1, SW25.1, SW26.1, SW27.1, SW28.1, SW29.1
- net SENSE2: now also SW24.1, SW25.1, SW26.1, SW27.1, SW28.1, SW29.1, SW31.1, SW32.1, SW35.1; no longer SW15.1, SW16.1, SW17.1, SW18.1, SW19.1, SW3.1
- net SENSE3: now also SW36.1, SW38.1, SW39.1, SW40.1, SW42.1, SW43.1, SW44.1, SW45.1, SW47.1, SW49.1; no longer SW20.1, SW31.1, SW4.1, SW5.1, SW6.1, SW7.1, SW8.1
- net DISCHAEGE0 renamed DISCHARGE0
- net DISCHAEGE1 renamed DISCHARGE1
- net DISCHAEGE2 renamed DISCHARGE2
- net DISCHAEGE3 renamed DISCHARGE3
- removed net SENSE4: SW10.1, SW21.1, SW22.1, SW32.1, SW43.1, SW9.1
- removed net SENSE5: SW11.1, SW12.1, SW23.1, SW40.1, SW42.1, SW44.1, SW47.1
- new net MUX0_D10: R53.1, U4.21 (Y10)
- new net MUX0_D11: R43.1, U4.20 (Y11)
- new net MUX0_D12: R52.1, U4.19 (Y12)
- new net MUX0_D13: R42.1, U4.18 (Y13)
- new net MUX0_D14: R51.1, U4.17 (Y14)
- new net MUX0_D15: R41.1, U4.16 (Y15)
- new net MUX0_D8: R54.1, U4.23 (Y8)
- new net MUX0_D9: R44.1, U4.22 (Y9)
- new net MUX1_D10: R63.1, U5.21 (Y10)
- new net MUX1_D11: R48.1, U5.20 (Y11)
- new net MUX1_D12: R62.1, U5.19 (Y12)
- new net MUX1_D13: R47.1, U5.18 (Y13)
- new net MUX1_D14: R61.1, U5.17 (Y14)
- new net MUX1_D15: R46.1, U5.16 (Y15)
- new net MUX1_D8: R64.1, U5.23 (Y8)
- new net MUX1_D9: R49.1, U5.22 (Y9)
- new net MUX2_D10: R73.1, U6.21 (Y10)
- new net MUX2_D11: R58.1, U6.20 (Y11)
- new net MUX2_D12: R72.1, U6.19 (Y12)
- new net MUX2_D13: R57.1, U6.18 (Y13)
- new net MUX2_D14: R71.1, U6.17 (Y14)
- new net MUX2_D15: R56.1, U6.16 (Y15)
- new net MUX2_D8: R74.1, U6.23 (Y8)
- new net MUX2_D9: R59.1, U6.22 (Y9)
- new net MUX3_D10: R78.1, U7.21 (Y10)
- new net MUX3_D11: R68.1, U7.20 (Y11)
- new net MUX3_D12: R77.1, U7.19 (Y12)
- new net MUX3_D13: R67.1, U7.18 (Y13)
- new net MUX3_D14: R76.1, U7.17 (Y14)
- new net MUX3_D15: R66.1, U7.16 (Y15)
- new net MUX3_D8: R79.1, U7.23 (Y8)
- new net MUX3_D9: R69.1, U7.22 (Y9)
- new net MUX_S3: U4.13 (A3), U5.13 (A3), U6.13 (A3), U7.13 (A3)
Other:
- moved on the sheet: C10, C11, C12, C18, C19, C20, C21, C22, C23, C24, C25, C9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

Commit message: 27.04.2026
Parts:
- SW1, SW2, SW3, SW35, SW38, SW39: footprint Kicad footprints:ecs_pad_1U_hybrid_hotswap_V3_switched_sides -> Kicad footprints:ecs_pad_1U_hybrid_hotswap_V3
- SW10, SW11, SW12, SW18, SW19, SW20, SW21, SW22, SW32, SW4, SW5: footprint Kicad footprints:ecs_pad_1U_hybrid_hotswap_V3 -> Kicad footprints:ecs_pad_1U_hybrid_hotswap_V3_switched_sides
Connections:
- net SENSE0: now also SW24.1, SW25.1, SW26.1, SW27.1, SW35.1, SW36.1, SW38.1, SW39.1, SW45.1, SW49.1; no longer SW10.1, SW11.1, SW12.1, SW2.1, SW23.1, SW3.1, SW4.1, SW5.1, SW6.1, SW7.1, SW8.1, SW9.1
- net SENSE1: now also SW2.1, SW28.1, SW3.1, SW4.1, SW5.1; no longer SW18.1, SW19.1, SW20.1, SW21.1, SW22.1
- net SENSE2: now also SW18.1, SW19.1, SW20.1, SW21.1, SW6.1, SW7.1, SW8.1, SW9.1; no longer SW24.1, SW25.1, SW26.1, SW27.1, SW28.1, SW32.1, SW35.1
- net SENSE3: now also SW10.1, SW11.1, SW12.1, SW22.1, SW23.1, SW32.1; no longer SW36.1, SW38.1, SW39.1, SW45.1, SW49.1

Commit message: 28.04.2026
Parts:
- SW18, SW19, SW20, SW21, SW40, SW42, SW6, SW7: footprint Kicad footprints:ecs_pad_1U_hybrid_hotswap_V3_switched_sides -> Kicad footprints:ecs_pad_1U_hybrid_hotswap_V3
- SW8, SW9: footprint Kicad footprints:ecs_pad_1U_hybrid_hotswap_V3 -> Kicad footprints:ecs_pad_1U_hybrid_hotswap_V3_switched_sides
Connections:
- net +3.3VA: no longer C10.1, C11.1, C12.1, C9.1, U4.24 (VDD), U5.24 (VDD), U6.24 (VDD), U7.24 (VDD)
- new net +3.3V: C10.1, C11.1, C12.1, C9.1, U4.24 (VDD), U5.24 (VDD), U6.24 (VDD), U7.24 (VDD)

Commit message: 29.04.2026
Connections:
- net MUX0_D10: now also SW26.2
- net MUX0_D11: now also SW25.2
- net MUX0_D12: now also SW24.2
- net MUX0_D13: now also SW35.2
- net MUX0_D14: now also SW36.2
- net MUX0_D15: now also SW45.2
- net MUX0_D5: now also SW38.2
- net MUX0_D6: now also SW49.2
- net MUX0_D7: now also SW39.2
- net MUX0_D9: now also SW27.2
- net MUX1_D0: now also SW4.2
- net MUX1_D1: now also SW3.2
- net MUX1_D13: now also SW28.2
- net MUX1_D14: now also SW17.2
- net MUX1_D15: now also SW5.2
- net MUX1_D2: now also SW2.2
- net MUX1_D3: now also SW1.2
- net MUX1_D4: now also SW13.2
- net MUX1_D5: now also SW14.2
- net MUX1_D6: now also SW15.2
- net MUX1_D7: now also SW16.2
- net MUX2_D6: now also SW29.2
- net MUX2_D7: now also SW30.2
- net MUX3_D0: now also SW44.2
- net MUX3_D10: now also SW11.2
- net MUX3_D11: now also SW32.2
- net MUX3_D12: now also SW40.2
- net MUX3_D13: now also SW47.2
- net MUX3_D14: now also SW42.2
- net MUX3_D15: now also SW43.2
- net MUX3_D6: now also SW12.2
- net MUX3_D7: now also SW23.2
- net MUX3_D8: now also SW22.2
- net MUX3_D9: now also SW10.2

Commit message: 30.04.2026
Parts:
- SW18, SW19, SW20, SW21: footprint Kicad footprints:ecs_pad_1U_hybrid_hotswap_V3 -> Kicad footprints:ecs_pad_1U_hybrid_hotswap_V3_switched_sides
Connections:
- net MUX1_D15: no longer SW5.2
- net MUX1_D7: now also SW5.2; no longer SW16.2
- net MUX1_D8: now also SW16.2
- net MUX2_D10: now also SW31.2
- net MUX2_D11: now also SW9.2
- net MUX2_D12: now also SW8.2
- net MUX2_D13: now also SW21.2
- net MUX2_D2: now also SW19.2
- net MUX2_D3: now also SW18.2
- net MUX2_D4: now also SW7.2
- net MUX2_D5: now also SW6.2
- net MUX2_D8: now also SW20.2
Changed lines of the file:
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@@
 	)
 	(junction
+		(at 392.43 72.39)
+		(diameter 0)
+		(color 0 0 0 0)
+	)
+	(junction
 		(at 172.72 264.16)
 		(diameter 0)
@@
 	)
 	(junction
-		(at 392.43 72.39)
-		(diameter 0)
-		(color 0 0 0 0)
-	)
-	(junction
 		(at 266.7 179.07)
 		(diameter 0)
@@
 	(wire
 		(pts
-			(xy 392.43 73.66) (xy 392.43 72.39)
-		)
-		(stroke
-			(width 0)
-			(type default)
-		)
-	)
-	(wire
-		(pts
 			(xy 370.84 205.74) (xy 381 205.74)
 		)
@@
 	(wire
 		(pts
-			(xy 392.43 73.66) (xy 393.7 73.66)
-		)
-		(stroke
-			(width 0)
-			(type default)
-		)
-	)
-	(wire
-		(pts
 			(xy 104.14 153.67) (xy 82.55 153.67)
 		)
@@
 		)
 	)
+	(global_label "MUX2_D12"
+		(shape input)
+		(at 227.33 30.48 90)
+		(fields_autoplaced yes)
+		(effects
+			(font
+				(size 1.27 1.27)
+			)
+			(justify left)
+		)
+		(property "Intersheetrefs" "${INTERSHEET_REFS}"
+			(at 227.33 17.6373 90)
+			(effects
+				(font
+					(size 1.27 1.27)
+				)
+				(justify left)
+				(hide yes)
+			)
+		)
+	)
+	(global_label "MUX2_D3"
+		(shape input)
+		(at 191.77 48.26 90)
+		(fields_autoplaced yes)
+		(effects
+			(font
+				(size 1.27 1.27)
+			)
+			(justify left)
+		)
+		(property "Intersheetrefs" "${INTERSHEET_REFS}"
+			(at 191.77 36.6268 90)
+			(effects
+				(font
+					(size 1.27 1.27)
+				)
+				(justify left)
+				(hide yes)
+			)
+		)
+	)
 	(global_label "SENSE3"
 		(shape input)
@@
 		)
 	)
+	(global_label "MUX2_D13"
+		(shape input)
+		(at 248.92 48.26 90)
+		(fields_autoplaced yes)
+		(effects
+			(font
+				(size 1.27 1.27)
+			)
+			(justify left)
+		)
+		(property "Intersheetrefs" "${INTERSHEET_REFS}"
+			(at 248.92 35.4173 90)
+			(effects
+				(font
+					(size 1.27 1.27)
+				)
+				(justify left)
+				(hide yes)
+			)
+		)
+	)
 	(global_label "MUX1_D4"
 		(shape input)
@@
 		)
 	)
+	(global_label "MUX2_D2"
+		(shape input)
+		(at 210.82 48.26 90)
+		(fields_autoplaced yes)
+		(effects
+			(font
+				(size 1.27 1.27)
+			)
+			(justify left)
+		)
+		(property "Intersheetrefs" "${INTERSHEET_REFS}"
+			(at 210.82 36.6268 90)
+			(effects
+				(font
+					(size 1.27 1.27)
+				)
+				(justify left)
+				(hide yes)
+			)
+		)
+	)
 	(global_label "SENSE0"
 		(shape input)
@@
 		)
 	)
+	(global_label "MUX2_D5"
+		(shape input)
+		(at 189.23 30.48 90)
+		(fields_autoplaced yes)
+		(effects
+			(font
+				(size 1.27 1.27)
+			)
+			(justify left)
+		)
+		(property "Intersheetrefs" "${INTERSHEET_REFS}"
+			(at 189.23 18.8468 90)
+			(effects
+				(font
+					(size 1.27 1.27)
+				)
+				(justify left)
+				(hide yes)
+			)
+		)
+	)
 	(global_label "MUX2_D6"
 		(shape input)
@@
 		)
 	)
-	(global_label "MUX1_D15"
+	(global_label "MUX1_D8"
 		(shape input)
-		(at 170.18 30.48 90)
+		(at 153.67 48.26 90)
 		(fields_autoplaced yes)
 		(effects
@@
 		)
 		(property "Intersheetrefs" "${INTERSHEET_REFS}"
-			(at 170.18 17.6373 90)
+			(at 153.67 36.6268 90)
 			(effects
 				(font
@@
 		)
 	)
+	(global_label "MUX2_D11"
+		(shape input)
+		(at 246.38 30.48 90)
+		(fields_autoplaced yes)
+		(effects
+			(font
+				(size 1.27 1.27)
+			)
+			(justify left)
+		)
+		(property "Intersheetrefs" "${INTERSHEET_REFS}"
+			(at 246.38 17.6373 90)
+			(effects
+				(font
+					(size 1.27 1.27)
+				)
+				(justify left)
+				(hide yes)
+			)
+		)
+	)
 	(global_label "MUX_S0"
 		(shape input)
@@
 		)
 	)
-	(global_label "MUX1_D7"
-		(shape input)
-		(at 153.67 48.26 90)
-		(fields_autoplaced yes)
-		(effects
-			(font
-				(size 1.27 1.27)
-			)
-			(justify left)
-		)
-		(property "Intersheetrefs" "${INTERSHEET_REFS}"
-			(at 153.67 36.6268 90)
-			(effects
-				(font
-					(size 1.27 1.27)
-				)
-				(justify left)
-				(hide yes)
-			)
-		)
-	)
 	(global_label "SENSE1"
 		(shape input)
@@
 		)
 	)
+	(global_label "MUX2_D8"
+		(shape input)
+		(at 229.87 48.26 90)
+		(fields_autoplaced yes)
+		(effects
+			(font
+				(size 1.27 1.27)
+			)
+			(justify left)
+		)
+		(property "Intersheetrefs" "${INTERSHEET_REFS}"
+			(at 229.87 36.6268 90)
+			(effects
+				(font
+					(size 1.27 1.27)
+				)
+				(justify left)
+				(hide yes)
+			)
+		)
+	)
 	(global_label "MUX3_D0"
 		(shape input)
@@
 		)
 	)
+	(global_label "MUX2_D10"
+		(shape input)
+		(at 233.68 66.04 90)
+		(fields_autoplaced yes)
+		(effects
+			(font
+				(size 1.27 1.27)
+			)
+			(justify left)
+		)
+		(property "Intersheetrefs" "${INTERSHEET_REFS}"
+			(at 233.68 53.1973 90)
+			(effects
+				(font
+					(size 1.27 1.27)
+				)
+				(justify left)
+				(hide yes)
+			)
+		)
+	)
 	(global_label "MUX0_D10"
 		(shape input)
@@
 		)
 	)
+	(global_label "MUX2_D4"
+		(shape input)
+		(at 208.28 30.48 90)
+		(fields_autoplaced yes)
+		(effects
+			(font
+				(size 1.27 1.27)
+			)
+			(justify left)
+		)
+		(property "Intersheetrefs" "${INTERSHEET_REFS}"
+			(at 208.28 18.8468 90)
+			(effects
+				(font
+					(size 1.27 1.27)
+				)
+				(justify left)
+				(hide yes)
+			)
+		)
+	)
 	(global_label "MUX3_D14"
 		(shape input)
@@
 		)
 	)
+	(global_label "MUX1_D7"
+		(shape input)
+		(at 170.18 30.48 90)
+		(fields_autoplaced yes)
+		(effects
+			(font
+				(size 1.27 1.27)
+			)
+			(justify left)
+		)
+		(property "Intersheetrefs" "${INTERSHEET_REFS}"
+			(at 170.18 18.8468 90)
+			(effects
+				(font
+					(size 1.27 1.27)
+				)
+				(justify left)
+				(hide yes)
+			)
+		)
+	)
 	(global_label "MUX1_D2"
 		(shape input)
@@
 			)
 		)
-		(property "Footprint" "Kicad footprints:ecs_pad_1U_hybrid_hotswap_V3"
+		(property "Footprint" "Kicad footprints:ecs_pad_1U_hybrid_hotswap_V3_switched_sides"
 			(at 222.25 48.26 0)
 			(effects
@@
 	(symbol
 		(lib_id "power:GND")
-		(at 393.7 73.66 0)
+		(at 392.43 72.39 0)
 		(unit 1)
 		(exclude_from_sim no)
@@
 		(fields_autoplaced yes)
 		(property "Reference" "#PWR09"
-			(at 393.7 80.01 0)
+			(at 392.43 78.74 0)
 			(effects
 				(font
@@
 		)
 		(property "Value" "GND"
-			(at 393.7 78.74 0)
+			(at 392.43 77.47 0)
 			(effects
 				(font
@@
 		)
 		(property "Footprint" ""
-			(at 393.7 73.66 0)
+			(at 392.43 72.39 0)
 			(effects
 				(font
@@
 		)
 		(property "Datasheet" ""
-			(at 393.7 73.66 0)
+			(at 392.43 72.39 0)
 			(effects
 				(font
@@
 		)
 		(property "Description" "Power symbol creates a global label with name \"GND\" , ground"
-			(at 393.7 73.66 0)
+			(at 392.43 72.39 0)
 			(effects
 				(font
@@
 			)
 		)
-		(property "Footprint" "Kicad footprints:ecs_pad_1U_hybrid_hotswap_V3"
+		(property "Footprint" "Kicad footprints:ecs_pad_1U_hybrid_hotswap_V3_switched_sides"
 			(at 203.2 48.26 0)
 			(effects
@@
 			)
 		)
-		(property "Footprint" "Kicad footprints:ecs_pad_1U_hybrid_hotswap_V3"
+		(property "Footprint" "Kicad footprints:ecs_pad_1U_hybrid_hotswap_V3_switched_sides"
 			(at 241.3 48.26 0)
 			(effects
@@
 			)
 		)
-		(property "Footprint" "Kicad footprints:ecs_pad_1U_hybrid_hotswap_V3"
+		(property "Footprint" "Kicad footprints:ecs_pad_1U_hybrid_hotswap_V3_switched_sides"
 			(at 184.15 48.26 0)
 			(effects

Commit message: 17.05.2026
Parts:
- SW13, SW14, SW15, SW16, SW17, SW38, SW39: footprint Kicad footprints:ecs_pad_1U_hybrid_hotswap_V3 -> Kicad footprints:ecs_pad_1U_hybrid_hotswap_V3_switched_sides
- SW24, SW25, SW32: footprint Kicad footprints:ecs_pad_1U_hybrid_hotswap_V3_switched_sides -> Kicad footprints:ecs_pad_1U_hybrid_hotswap_V3
Connections:
- net SENSE0: now also SW1.1, SW13.1, SW14.1, SW15.1, SW2.1, SW3.1; no longer SW26.1, SW27.1, SW38.1, SW39.1, SW49.1
- net SENSE1: now also SW18.1, SW26.1, SW27.1, SW29.1, SW38.1, SW6.1; no longer SW1.1, SW13.1, SW14.1, SW15.1, SW2.1, SW3.1
- net SENSE2: now also SW39.1, SW49.1; no longer SW18.1, SW29.1, SW6.1

Commit message: 18.05.2026
Parts:
- SW1, SW2, SW24, SW25, SW3, SW32, SW35, SW40, SW42, SW6: footprint Kicad footprints:ecs_pad_1U_hybrid_hotswap_V3 -> Kicad footprints:ecs_pad_1U_hybrid_hotswap_V3_switched_sides
Changed lines of the file:
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@@
 			)
 		)
-		(property "Footprint" "Kicad footprints:ecs_pad_1U_hybrid_hotswap_V3"
+		(property "Footprint" "Kicad footprints:ecs_pad_1U_hybrid_hotswap_V3_switched_sides"
 			(at 124.46 30.48 0)
 			(effects
@@
 			)
 		)
-		(property "Footprint" "Kicad footprints:ecs_pad_1U_hybrid_hotswap_V3"
+		(property "Footprint" "Kicad footprints:ecs_pad_1U_hybrid_hotswap_V3_switched_sides"
 			(at 92.71 66.04 0)
 			(effects
@@
 			)
 		)
-		(property "Footprint" "Kicad footprints:ecs_pad_1U_hybrid_hotswap_V3"
+		(property "Footprint" "Kicad footprints:ecs_pad_1U_hybrid_hotswap_V3_switched_sides"
 			(at 245.11 66.04 0)
 			(effects
@@
 			)
 		)
-		(property "Footprint" "Kicad footprints:ecs_pad_1U_hybrid_hotswap_V3"
+		(property "Footprint" "Kicad footprints:ecs_pad_1U_hybrid_hotswap_V3_switched_sides"
 			(at 232.41 83.82 0)
 			(effects
@@
 			)
 		)
-		(property "Footprint" "Kicad footprints:ecs_pad_1U_hybrid_hotswap_V3"
+		(property "Footprint" "Kicad footprints:ecs_pad_1U_hybrid_hotswap_V3_switched_sides"
 			(at 111.76 66.04 0)
 			(effects
@@
 			)
 		)
-		(property "Footprint" "Kicad footprints:ecs_pad_1U_hybrid_hotswap_V3"
+		(property "Footprint" "Kicad footprints:ecs_pad_1U_hybrid_hotswap_V3_switched_sides"
 			(at 270.51 83.82 0)
 			(effects
@@
 			)
 		)
-		(property "Footprint" "Kicad footprints:ecs_pad_1U_hybrid_hotswap_V3"
+		(property "Footprint" "Kicad footprints:ecs_pad_1U_hybrid_hotswap_V3_switched_sides"
 			(at 181.61 30.48 0)
 			(effects
@@
 			)
 		)
-		(property "Footprint" "Kicad footprints:ecs_pad_1U_hybrid_hotswap_V3"
+		(property "Footprint" "Kicad footprints:ecs_pad_1U_hybrid_hotswap_V3_switched_sides"
 			(at 86.36 30.48 0)
 			(effects
@@
 			)
 		)
-		(property "Footprint" "Kicad footprints:ecs_pad_1U_hybrid_hotswap_V3"
+		(property "Footprint" "Kicad footprints:ecs_pad_1U_hybrid_hotswap_V3_switched_sides"
 			(at 105.41 30.48 0)
 			(effects
@@
 			)
 		)
-		(property "Footprint" "Kicad footprints:ecs_pad_1U_hybrid_hotswap_V3"
+		(property "Footprint" "Kicad footprints:ecs_pad_1U_hybrid_hotswap_V3_switched_sides"
 			(at 86.36 83.82 0)
 			(effects

Commit message: 19.05.2026
Connections:
- net MUX0_IN: no longer U5.1 (Z), U6.1 (Z), U7.1 (Z)
- new net MUX1_IN: U5.1 (Z)
- new net MUX2_IN: U6.1 (Z)
- new net MUX3_IN: U7.1 (Z)
