File: Romashka EC non-matrix/Logic.kicad_sch (KiCad schematic)
At the start: 149 parts, among them SW1 EC_SW, SW10 EC_SW, SW11 EC_SW, SW12 EC_SW, SW13 EC_SW, SW14 EC_SW, SW15 EC_SW, SW16 EC_SW, SW17 EC_SW, SW18 EC_SW, SW19 EC_SW, SW2 EC_SW, SW20 EC_SW, SW21 EC_SW, SW22 EC_SW, SW23 EC_SW, SW24 EC_SW, SW25 EC_SW, SW26 EC_SW, SW27 EC_SW, SW28 EC_SW, SW29 EC_SW, SW3 EC_SW, SW30 EC_SW, SW31 EC_SW, SW32 EC_SW, SW33 EC_SW, SW34 EC_SW, SW35 EC_SW, SW36 EC_SW, SW37 EC_SW, SW38 EC_SW, SW39 EC_SW, SW4 EC_SW, SW40 EC_SW, SW41 EC_SW, SW42 EC_SW, SW43 EC_SW, SW44 EC_SW, SW45 EC_SW, SW46 EC_SW, SW47 EC_SW, SW48 EC_SW, SW49 EC_SW, SW5 EC_SW, SW6 EC_SW, SW7 EC_SW, SW8 EC_SW, SW9 EC_SW, U10 TLV9061xDBV, U11 TLV9061xDBV, U4 HEF4067BTT, U5 HEF4067BTT, U6 HEF4067BTT, U7 HEF4067BTT, U8 TLV9061xDBV, U9 TLV9061xDBV

Commit message: 19.05.2026
Parts:
- removed R13, R14, R17, R21, R22, R33, R34, R37, R40, R44, R49, R54, R64, R69, R79, R8, R9: 100K, Resistor_SMD:R_0603_1608Metric, symbol Device:R_Small
- SW1, SW2, SW3, SW32, SW35, SW40, SW42, SW6: footprint Kicad footprints:ecs_pad_1U_hybrid_hotswap_V3_switched_sides -> Kicad footprints:ecs_pad_1U_hybrid_hotswap_V3
Connections:
- net MUX0_D3 is gone; now on net GND: U4.6 (Y3)
- net MUX0_D4 is gone; now on net GND: U4.5 (Y4)
- net MUX0_D8 is gone; now on net GND: U4.23 (Y8)
- net MUX1_D9 is gone; now on net GND: U5.22 (Y9)
- net GND: now also U4.22 (Y9), U4.4 (Y5), U5.23 (Y8), U5.4 (Y5), U5.5 (Y4), U5.6 (Y3), U6.22 (Y9), U6.23 (Y8), U6.4 (Y5), U6.5 (Y4), U6.6 (Y3), U7.22 (Y9), U7.23 (Y8), U7.4 (Y5), U7.5 (Y4), U7.6 (Y3)
- net MUX0_D0: now also SW35.2
- net MUX0_D1: now also SW24.2
- net MUX0_D10: now also SW14.2; no longer SW26.2
- net MUX0_D11: now also SW15.2; no longer SW25.2
- net MUX0_D12: now also SW3.2; no longer SW24.2
- net MUX0_D13: now also SW2.2; no longer SW35.2
- net MUX0_D14: now also SW1.2; no longer SW36.2
- net MUX0_D15: now also SW13.2; no longer SW45.2
- net MUX0_D2: now also SW36.2
- net MUX0_D6: now also SW45.2
- net MUX0_D7: now also SW25.2
- net MUX1_D0: now also SW26.2; no longer SW4.2
- net MUX1_D1: now also SW38.2; no longer SW3.2
- net MUX1_D10: now also SW17.2
- net MUX1_D11: now also SW18.2
- net MUX1_D12: now also SW6.2
- net MUX1_D13: now also SW5.2; no longer SW28.2
- net MUX1_D14: now also SW4.2; no longer SW17.2
- net MUX1_D15: now also SW16.2
- net MUX1_D2: now also SW27.2; no longer SW2.2
- net MUX1_D6: now also SW28.2; no longer SW15.2
- net MUX1_D7: now also SW29.2; no longer SW5.2
- net MUX2_D4: no longer U6.5 (Y4)
- net MUX2_D6: no longer SW29.2
- net MUX2_D8: no longer R74.1, U6.23 (Y8)
- net MUX3_D0: no longer SW44.2
- net MUX3_D10: now also SW23.2; no longer SW11.2
- net MUX3_D11: now also SW12.2; no longer SW32.2
- net MUX3_D12: now also SW11.2; no longer SW40.2
- net MUX3_D13: now also SW10.2; no longer SW47.2
- net MUX3_D14: now also SW22.2; no longer SW42.2
- net MUX3_D15: no longer SW43.2
- net MUX3_D2: now also SW32.2
- net MUX3_D3: now also SW40.2; no longer U7.6 (Y3)
- net MUX3_D4: now also SW47.2; no longer U7.5 (Y4)
- net MUX3_D5: now also SW43.2; no longer U7.4 (Y5)
- net MUX3_D6: now also SW42.2; no longer SW12.2
- net MUX3_D7: now also SW44.2; no longer SW23.2
- removed net MUX0_D5: SW38.2, U4.4 (Y5)
- removed net MUX0_D9: SW27.2, U4.22 (Y9)
- removed net MUX1_D3: SW1.2, U5.6 (Y3)
- removed net MUX1_D4: R29.2, SW13.2, U5.5 (Y4)
- removed net MUX1_D5: SW14.2, U5.4 (Y5)
- removed net MUX1_D8: SW16.2, U5.23 (Y8)
- removed net MUX2_D3: SW18.2, U6.6 (Y3)
- removed net MUX2_D5: SW6.2, U6.4 (Y5)
- net MUX2_D9: no longer names the net of R59.1
- net MUX2_D9: no longer U6.22 (Y9)
- removed net MUX3_D8: SW22.2, U7.23 (Y8)
- removed net MUX3_D9: SW10.2, U7.22 (Y9)

Commit message: 20.05.2026
Parts:
- SW24, SW25: footprint Kicad footprints:ecs_pad_1U_hybrid_hotswap_V3_switched_sides -> Kicad footprints:ecs_pad_1U_hybrid_hotswap_V3
Connections:
- net MUX2_D4 is gone; now on net MUX2_D14: SW7.2
- net MUX2_D8 is gone; now on net MUX2_D10: SW20.2
- net MUX3_D3 is gone; now on net MUX3_D1: SW40.2
- net MUX3_D4 is gone; now on net MUX3_D2: SW47.2
- net MUX0_D6: no longer SW49.2
- net MUX0_D7: no longer SW39.2
- net MUX2_D1: now also SW30.2
- net MUX2_D10: no longer SW31.2
- net MUX2_D11: now also SW21.2; no longer SW9.2
- net MUX2_D12: now also SW9.2; no longer SW8.2
- net MUX2_D13: now also SW8.2; no longer SW21.2
- net MUX2_D15: now also SW19.2
- net MUX2_D2: now also SW49.2; no longer SW19.2
- net MUX2_D6: now also SW39.2
- net MUX2_D7: now also SW31.2; no longer SW30.2
- net MUX3_D0: now also SW32.2
- net MUX3_D2: no longer SW32.2

Commit message: 22.05.2026
Connections:
- net MUX2_D10: now also SW21.2; no longer SW20.2
- net MUX2_D11: now also SW20.2; no longer SW21.2

Commit message: 25.05.2026
Connections:
- net +3.3VA is gone; now on net +3.3V: C18.2, C19.2, C20.2, C21.2, U10.5 (V+), U11.5 (V+), U8.5 (V+), U9.5 (V+)

Commit message: 25.05.2026
Parts:
- SW24, SW25: footprint Kicad footprints:ecs_pad_1U_hybrid_hotswap_V3 -> Kicad footprints:ecs_pad_1U_hybrid_hotswap_V3_switched_sides
Changed lines of the file:
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@@
 			)
 		)
-		(property "Footprint" "Kicad footprints:ecs_pad_1U_hybrid_hotswap_V3"
+		(property "Footprint" "Kicad footprints:ecs_pad_1U_hybrid_hotswap_V3_switched_sides"
 			(at 92.71 66.04 0)
 			(effects
@@
 			)
 		)
-		(property "Footprint" "Kicad footprints:ecs_pad_1U_hybrid_hotswap_V3"
+		(property "Footprint" "Kicad footprints:ecs_pad_1U_hybrid_hotswap_V3_switched_sides"
 			(at 111.76 66.04 0)
 			(effects

Commit message: 26.05.2026
Parts:
- SW32: footprint Kicad footprints:ecs_pad_1U_hybrid_hotswap_V3 -> Kicad footprints:ecs_pad_1U_hybrid_hotswap_V3_switched_sides
Changed lines of the file:
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@@
 			)
 		)
-		(property "Footprint" "Kicad footprints:ecs_pad_1U_hybrid_hotswap_V3"
+		(property "Footprint" "Kicad footprints:ecs_pad_1U_hybrid_hotswap_V3_switched_sides"
 			(at 245.11 66.04 0)
 			(effects
