File: Romashka EC non-matrix/Logic.kicad_sch (KiCad schematic)
At the start: 132 parts, among them SW1 EC_SW, SW10 EC_SW, SW11 EC_SW, SW12 EC_SW, SW13 EC_SW, SW14 EC_SW, SW15 EC_SW, SW16 EC_SW, SW17 EC_SW, SW18 EC_SW, SW19 EC_SW, SW2 EC_SW, SW20 EC_SW, SW21 EC_SW, SW22 EC_SW, SW23 EC_SW, SW24 EC_SW, SW25 EC_SW, SW26 EC_SW, SW27 EC_SW, SW28 EC_SW, SW29 EC_SW, SW3 EC_SW, SW30 EC_SW, SW31 EC_SW, SW32 EC_SW, SW33 EC_SW, SW34 EC_SW, SW35 EC_SW, SW36 EC_SW, SW37 EC_SW, SW38 EC_SW, SW39 EC_SW, SW4 EC_SW, SW40 EC_SW, SW41 EC_SW, SW42 EC_SW, SW43 EC_SW, SW44 EC_SW, SW45 EC_SW, SW46 EC_SW, SW47 EC_SW, SW48 EC_SW, SW49 EC_SW, SW5 EC_SW, SW6 EC_SW, SW7 EC_SW, SW8 EC_SW, SW9 EC_SW, U10 TLV9061xDBV, U11 TLV9061xDBV, U4 HEF4067BTT, U5 HEF4067BTT, U6 HEF4067BTT, U7 HEF4067BTT, U8 TLV9061xDBV, U9 TLV9061xDBV

Commit message: 20.08.2026
Parts:
- SW1, SW2, SW3, SW33, SW34, SW35, SW40, SW41, SW42, SW46, SW48, SW6, SW7: footprint Kicad footprints:ecs_pad_1U_hybrid_hotswap_V3 -> FriedSoul_switches:ecs_pad_1U_hybrid_hotswap_V3
- SW10, SW11, SW12, SW13, SW14, SW15, SW16, SW17, SW18, SW19, SW20, SW21, SW22, SW23, SW24, SW25, SW26, SW27, SW28, SW29, SW30, SW31, SW32, SW38, SW39, SW4, SW5, SW8, SW9: footprint Kicad footprints:ecs_pad_1U_hybrid_hotswap_V3_switched_sides -> FriedSoul_switches:ecs_pad_1U_hybrid_hotswap_V3_switched_sides
- SW36, SW43, SW44, SW45, SW47: footprint Kicad footprints:ecs_pad_hybrid_hotswap_2.381_V3 -> FriedSoul_switches:ecs_pad_hybrid_hotswap_2.381_V3
- SW49: footprint Kicad footprints:ecs_pad_hybrid_hotswap_7.144_V3 -> FriedSoul_switches:ecs_pad_hybrid_hotswap_7.144_V3

Commit message: 20.08.2026
Parts:
- removed R59, R74: 100K, Resistor_SMD:R_0603_1608Metric, symbol Device:R_Small
Connections:
- net GND: no longer U4.15 (~{E}), U5.15 (~{E}), U6.15 (~{E}), U7.15 (~{E})
- new net MUX_EN: U4.15 (~{E}), U5.15 (~{E}), U6.15 (~{E}), U7.15 (~{E})
