File: Romashka EC non-matrix/Logic.kicad_sch (KiCad schematic)
At the start: 130 parts, among them SW1 EC_SW, SW10 EC_SW, SW11 EC_SW, SW12 EC_SW, SW13 EC_SW, SW14 EC_SW, SW15 EC_SW, SW16 EC_SW, SW17 EC_SW, SW18 EC_SW, SW19 EC_SW, SW2 EC_SW, SW20 EC_SW, SW21 EC_SW, SW22 EC_SW, SW23 EC_SW, SW24 EC_SW, SW25 EC_SW, SW26 EC_SW, SW27 EC_SW, SW28 EC_SW, SW29 EC_SW, SW3 EC_SW, SW30 EC_SW, SW31 EC_SW, SW32 EC_SW, SW33 EC_SW, SW34 EC_SW, SW35 EC_SW, SW36 EC_SW, SW37 EC_SW, SW38 EC_SW, SW39 EC_SW, SW4 EC_SW, SW40 EC_SW, SW41 EC_SW, SW42 EC_SW, SW43 EC_SW, SW44 EC_SW, SW45 EC_SW, SW46 EC_SW, SW47 EC_SW, SW48 EC_SW, SW49 EC_SW, SW5 EC_SW, SW6 EC_SW, SW7 EC_SW, SW8 EC_SW, SW9 EC_SW, U10 TLV9061xDBV, U11 TLV9061xDBV, U4 HEF4067BTT, U5 HEF4067BTT, U6 HEF4067BTT, U7 HEF4067BTT, U8 TLV9061xDBV, U9 TLV9061xDBV

Commit message: 21.08.2026
Parts:
- SW35: footprint FriedSoul_switches:ecs_pad_1U_hybrid_hotswap_V3 -> FriedSoul_switches:ecs_pad_1U_hybrid_hotswap_V3_switched_sides
- SW39: footprint FriedSoul_switches:ecs_pad_1U_hybrid_hotswap_V3_switched_sides -> FriedSoul_switches:ecs_pad_1U_hybrid_hotswap_V3
Connections:
- net SENSE0: now also SW38.1; no longer SW15.1
- net SENSE1: now also SW15.1; no longer SW38.1
Changed lines of the file:
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@@
 		)
 	)
-	(global_label "SENSE0"
-		(shape input)
-		(at 119.38 48.26 90)
-		(fields_autoplaced yes)
-		(effects
-			(font
-				(size 1.27 1.27)
-				(color 255 0 6 1)
-			)
-			(justify left)
-		)
-		(property "Intersheetrefs" "${INTERSHEET_REFS}"
-			(at 119.38 38.0178 90)
-			(effects
-				(font
-					(size 1.27 1.27)
-				)
-				(justify left)
-				(hide yes)
-			)
-		)
-	)
 	(global_label "SENSE3"
 		(shape input)
@@
 		)
 	)
-	(global_label "SENSE1"
-		(shape input)
-		(at 180.34 66.04 90)
-		(fields_autoplaced yes)
-		(effects
-			(font
-				(size 1.27 1.27)
-				(color 0 6 255 1)
-			)
-			(justify left)
-		)
-		(property "Intersheetrefs" "${INTERSHEET_REFS}"
-			(at 180.34 55.7978 90)
-			(effects
-				(font
-					(size 1.27 1.27)
-				)
-				(justify left)
-				(hide yes)
-			)
-		)
-	)
 	(global_label "MUX_S2"
 		(shape input)
@@
 		)
 	)
-	(global_label "SENSE1"
-		(shape input)
-		(at 176.53 48.26 90)
-		(fields_autoplaced yes)
-		(effects
-			(font
-				(size 1.27 1.27)
-				(color 0 6 255 1)
-			)
-			(justify left)
-		)
-		(property "Intersheetrefs" "${INTERSHEET_REFS}"
-			(at 176.53 38.0178 90)
-			(effects
-				(font
-					(size 1.27 1.27)
-				)
-				(justify left)
-				(hide yes)
-			)
-		)
-	)
 	(global_label "MUX0_D10"
 		(shape input)
@@
 		)
 	)
+	(global_label "SENSE2"
+		(shape input)
+		(at 189.23 83.82 90)
+		(fields_autoplaced yes)
+		(effects
+			(font
+				(size 1.27 1.27)
+				(color 255 123 4 1)
+			)
+			(justify left)
+		)
+		(property "Intersheetrefs" "${INTERSHEET_REFS}"
+			(at 189.23 73.5778 90)
+			(effects
+				(font
+					(size 1.27 1.27)
+				)
+				(justify left)
+				(hide yes)
+			)
+		)
+	)
 	(global_label "SENSE0"
 		(shape input)
@@
 		)
 	)
-	(global_label "SENSE2"
-		(shape input)
-		(at 189.23 83.82 90)
-		(fields_autoplaced yes)
-		(effects
-			(font
-				(size 1.27 1.27)
-				(color 255 123 4 1)
-			)
-			(justify left)
-		)
-		(property "Intersheetrefs" "${INTERSHEET_REFS}"
-			(at 189.23 73.5778 90)
-			(effects
-				(font
-					(size 1.27 1.27)
-				)
-				(justify left)
-				(hide yes)
-			)
-		)
-	)
 	(global_label "MUX2_D2"
 		(shape input)
@@
 		)
 	)
-	(global_label "SENSE1"
-		(shape input)
-		(at 123.19 66.04 90)
-		(fields_autoplaced yes)
-		(effects
-			(font
-				(size 1.27 1.27)
-				(color 0 6 255 1)
-			)
-			(justify left)
-		)
-		(property "Intersheetrefs" "${INTERSHEET_REFS}"
-			(at 123.19 55.7978 90)
-			(effects
-				(font
-					(size 1.27 1.27)
-				)
-				(justify left)
-				(hide yes)
-			)
-		)
-	)
 	(global_label "MUX2_D1"
 		(shape input)
@@
 		)
 	)
-	(global_label "SENSE1"
-		(shape input)
-		(at 149.86 83.82 90)
-		(fields_autoplaced yes)
-		(effects
-			(font
-				(size 1.27 1.27)
-				(color 0 6 255 1)
-			)
-			(justify left)
-		)
-		(property "Intersheetrefs" "${INTERSHEET_REFS}"
-			(at 149.86 73.5778 90)
-			(effects
-				(font
-					(size 1.27 1.27)
-				)
-				(justify left)
-				(hide yes)
-			)
-		)
-	)
 	(global_label "SENSE0"
 		(shape input)
@@
 		)
 	)
+	(global_label "SENSE1"
+		(shape input)
+		(at 119.38 48.26 90)
+		(fields_autoplaced yes)
+		(effects
+			(font
+				(size 1.27 1.27)
+				(color 0 6 255 1)
+			)
+			(justify left)
+		)
+		(property "Intersheetrefs" "${INTERSHEET_REFS}"
+			(at 119.38 38.0178 90)
+			(effects
+				(font
+					(size 1.27 1.27)
+				)
+				(justify left)
+				(hide yes)
+			)
+		)
+	)
 	(global_label "MUX3_D7"
 		(shape input)
@@
 		)
 	)
+	(global_label "SENSE1"
+		(shape input)
+		(at 180.34 66.04 90)
+		(fields_autoplaced yes)
+		(effects
+			(font
+				(size 1.27 1.27)
+				(color 0 6 255 1)
+			)
+			(justify left)
+		)
+		(property "Intersheetrefs" "${INTERSHEET_REFS}"
+			(at 180.34 55.7978 90)
+			(effects
+				(font
+					(size 1.27 1.27)
+				)
+				(justify left)
+				(hide yes)
+			)
+		)
+	)
 	(global_label "MUX2_D0"
 		(shape input)
@@
 		)
 	)
+	(global_label "SENSE1"
+		(shape input)
+		(at 176.53 48.26 90)
+		(fields_autoplaced yes)
+		(effects
+			(font
+				(size 1.27 1.27)
+				(color 0 6 255 1)
+			)
+			(justify left)
+		)
+		(property "Intersheetrefs" "${INTERSHEET_REFS}"
+			(at 176.53 38.0178 90)
+			(effects
+				(font
+					(size 1.27 1.27)
+				)
+				(justify left)
+				(hide yes)
+			)
+		)
+	)
 	(global_label "MUX2_D15"
 		(shape input)
@@
 		)
 	)
+	(global_label "SENSE1"
+		(shape input)
+		(at 123.19 66.04 90)
+		(fields_autoplaced yes)
+		(effects
+			(font
+				(size 1.27 1.27)
+				(color 0 6 255 1)
+			)
+			(justify left)
+		)
+		(property "Intersheetrefs" "${INTERSHEET_REFS}"
+			(at 123.19 55.7978 90)
+			(effects
+				(font
+					(size 1.27 1.27)
+				)
+				(justify left)
+				(hide yes)
+			)
+		)
+	)
+	(global_label "SENSE0"
+		(shape input)
+		(at 149.86 83.82 90)
+		(fields_autoplaced yes)
+		(effects
+			(font
+				(size 1.27 1.27)
+				(color 255 0 6 1)
+			)
+			(justify left)
+		)
+		(property "Intersheetrefs" "${INTERSHEET_REFS}"
+			(at 149.86 73.5778 90)
+			(effects
+				(font
+					(size 1.27 1.27)
+				)
+				(justify left)
+				(hide yes)
+			)
+		)
+	)
 	(global_label "MUX0_D14"
 		(shape input)
@@
 		)
 	)
+	(global_label "SENSE2"
+		(shape input)
+		(at 386.08 100.33 90)
+		(fields_autoplaced yes)
+		(effects
+			(font
+				(size 1.27 1.27)
+				(color 255 123 4 1)
+			)
+			(justify left)
+		)
+		(property "Intersheetrefs" "${INTERSHEET_REFS}"
+			(at 386.08 90.0878 90)
+			(effects
+				(font
+					(size 1.27 1.27)
+				)
+				(justify left)
+				(hide yes)
+			)
+		)
+	)
 	(global_label "SENSE0"
 		(shape input)
@@
 		)
 	)
-	(global_label "SENSE2"
-		(shape input)
-		(at 386.08 100.33 90)
-		(fields_autoplaced yes)
-		(effects
-			(font
-				(size 1.27 1.27)
-				(color 255 123 4 1)
-			)
-			(justify left)
-		)
-		(property "Intersheetrefs" "${INTERSHEET_REFS}"
-			(at 386.08 90.0878 90)
-			(effects
-				(font
-					(size 1.27 1.27)
-				)
-				(justify left)
-				(hide yes)
-			)
-		)
-	)
 	(global_label "SENSE3"
 		(shape input)
@@
 			)
 		)
-		(property "Footprint" "FriedSoul_switches:ecs_pad_1U_hybrid_hotswap_V3_switched_sides"
+		(property "Footprint" "FriedSoul_switches:ecs_pad_1U_hybrid_hotswap_V3"
 			(at 196.85 83.82 0)
 			(effects
@@
 			)
 		)
-		(property "Footprint" "FriedSoul_switches:ecs_pad_1U_hybrid_hotswap_V3"
+		(property "Footprint" "FriedSoul_switches:ecs_pad_1U_hybrid_hotswap_V3_switched_sides"
 			(at 86.36 83.82 0)
 			(effects

Commit message: 24.08.2026
Parts:
- SW39: footprint FriedSoul_switches:ecs_pad_1U_hybrid_hotswap_V3 -> FriedSoul_switches:ecs_pad_1U_hybrid_hotswap_V3_switched_sides
Connections:
- net SENSE0: now also SW39.1, SW49.1; no longer SW14.1, SW25.1, SW3.1
- net SENSE1: now also SW14.1, SW25.1, SW3.1; no longer SW18.1, SW28.1, SW29.1
- net SENSE2: now also SW18.1, SW28.1, SW29.1; no longer SW39.1, SW49.1
Changed lines of the file:
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@@
 		)
 	)
-	(global_label "SENSE1"
+	(global_label "MUX0_D1"
 		(shape input)
-		(at 161.29 66.04 90)
+		(at 104.14 146.05 0)
 		(fields_autoplaced yes)
 		(effects
 			(font
 				(size 1.27 1.27)
-				(color 0 6 255 1)
 			)
 			(justify left)
 		)
 		(property "Intersheetrefs" "${INTERSHEET_REFS}"
-			(at 161.29 55.7978 90)
+			(at 115.7732 146.05 0)
 			(effects
 				(font
@@
 		)
 	)
-	(global_label "MUX0_D1"
+	(global_label "SENSE0"
 		(shape input)
-		(at 104.14 146.05 0)
+		(at 189.23 83.82 90)
 		(fields_autoplaced yes)
 		(effects
 			(font
 				(size 1.27 1.27)
+				(color 255 0 6 1)
 			)
 			(justify left)
 		)
 		(property "Intersheetrefs" "${INTERSHEET_REFS}"
-			(at 115.7732 146.05 0)
+			(at 189.23 73.5778 90)
 			(effects
 				(font
@@
 		)
 	)
-	(global_label "SENSE0"
-		(shape input)
-		(at 116.84 30.48 90)
-		(fields_autoplaced yes)
-		(effects
-			(font
-				(size 1.27 1.27)
-				(color 255 0 6 1)
-			)
-			(justify left)
-		)
-		(property "Intersheetrefs" "${INTERSHEET_REFS}"
-			(at 116.84 20.2378 90)
-			(effects
-				(font
-					(size 1.27 1.27)
-				)
-				(justify left)
-				(hide yes)
-			)
-		)
-	)
 	(global_label "SENSE2"
 		(shape input)
@@
 		)
 	)
-	(global_label "SENSE2"
-		(shape input)
-		(at 189.23 83.82 90)
-		(fields_autoplaced yes)
-		(effects
-			(font
-				(size 1.27 1.27)
-				(color 255 123 4 1)
-			)
-			(justify left)
-		)
-		(property "Intersheetrefs" "${INTERSHEET_REFS}"
-			(at 189.23 73.5778 90)
-			(effects
-				(font
-					(size 1.27 1.27)
-				)
-				(justify left)
-				(hide yes)
-			)
-		)
-	)
-	(global_label "SENSE0"
-		(shape input)
-		(at 100.33 48.26 90)
-		(fields_autoplaced yes)
-		(effects
-			(font
-				(size 1.27 1.27)
-				(color 255 0 6 1)
-			)
-			(justify left)
-		)
-		(property "Intersheetrefs" "${INTERSHEET_REFS}"
-			(at 100.33 38.0178 90)
-			(effects
-				(font
-					(size 1.27 1.27)
-				)
-				(justify left)
-				(hide yes)
-			)
-		)
-	)
 	(global_label "MUX3_D1"
 		(shape input)
@@
 		)
 	)
-	(global_label "SENSE0"
-		(shape input)
-		(at 104.14 66.04 90)
-		(fields_autoplaced yes)
-		(effects
-			(font
-				(size 1.27 1.27)
-				(color 255 0 6 1)
-			)
-			(justify left)
-		)
-		(property "Intersheetrefs" "${INTERSHEET_REFS}"
-			(at 104.14 55.7978 90)
-			(effects
-				(font
-					(size 1.27 1.27)
-				)
-				(justify left)
-				(hide yes)
-			)
-		)
-	)
 	(global_label "SENSE2"
 		(shape input)
@@
 		)
 	)
+	(global_label "SENSE0"
+		(shape input)
+		(at 386.08 100.33 90)
+		(fields_autoplaced yes)
+		(effects
+			(font
+				(size 1.27 1.27)
+				(color 255 0 6 1)
+			)
+			(justify left)
+		)
+		(property "Intersheetrefs" "${INTERSHEET_REFS}"
+			(at 386.08 90.0878 90)
+			(effects
+				(font
+					(size 1.27 1.27)
+				)
+				(justify left)
+				(hide yes)
+			)
+		)
+	)
+	(global_label "SENSE2"
+		(shape input)
+		(at 180.34 66.04 90)
+		(fields_autoplaced yes)
+		(effects
+			(font
+				(size 1.27 1.27)
+				(color 255 123 4 1)
+			)
+			(justify left)
+		)
+		(property "Intersheetrefs" "${INTERSHEET_REFS}"
+			(at 180.34 55.7978 90)
+			(effects
+				(font
+					(size 1.27 1.27)
+				)
+				(justify left)
+				(hide yes)
+			)
+		)
+	)
 	(global_label "SENSE2"
 		(shape input)
@@
 		)
 	)
+	(global_label "SENSE2"
+		(shape input)
+		(at 176.53 48.26 90)
+		(fields_autoplaced yes)
+		(effects
+			(font
+				(size 1.27 1.27)
+				(color 255 123 4 1)
+			)
+			(justify left)
+		)
+		(property "Intersheetrefs" "${INTERSHEET_REFS}"
+			(at 176.53 38.0178 90)
+			(effects
+				(font
+					(size 1.27 1.27)
+				)
+				(justify left)
+				(hide yes)
+			)
+		)
+	)
 	(global_label "MUX2_D2"
 		(shape input)
@@
 		)
 	)
-	(global_label "SENSE1"
-		(shape input)
-		(at 180.34 66.04 90)
-		(fields_autoplaced yes)
-		(effects
-			(font
-				(size 1.27 1.27)
-				(color 0 6 255 1)
-			)
-			(justify left)
-		)
-		(property "Intersheetrefs" "${INTERSHEET_REFS}"
-			(at 180.34 55.7978 90)
-			(effects
-				(font
-					(size 1.27 1.27)
-				)
-				(justify left)
-				(hide yes)
-			)
-		)
-	)
 	(global_label "MUX2_D0"
 		(shape input)
@@
 		)
 	)
-	(global_label "SENSE1"
-		(shape input)
-		(at 176.53 48.26 90)
-		(fields_autoplaced yes)
-		(effects
-			(font
-				(size 1.27 1.27)
-				(color 0 6 255 1)
-			)
-			(justify left)
-		)
-		(property "Intersheetrefs" "${INTERSHEET_REFS}"
-			(at 176.53 38.0178 90)
-			(effects
-				(font
-					(size 1.27 1.27)
-				)
-				(justify left)
-				(hide yes)
-			)
-		)
-	)
 	(global_label "MUX2_D15"
 		(shape input)
@@
 		)
 	)
+	(global_label "SENSE2"
+		(shape input)
+		(at 161.29 66.04 90)
+		(fields_autoplaced yes)
+		(effects
+			(font
+				(size 1.27 1.27)
+				(color 255 123 4 1)
+			)
+			(justify left)
+		)
+		(property "Intersheetrefs" "${INTERSHEET_REFS}"
+			(at 161.29 55.7978 90)
+			(effects
+				(font
+					(size 1.27 1.27)
+				)
+				(justify left)
+				(hide yes)
+			)
+		)
+	)
 	(global_label "MUX3_D2"
 		(shape input)
@@
 		)
 	)
+	(global_label "SENSE1"
+		(shape input)
+		(at 104.14 66.04 90)
+		(fields_autoplaced yes)
+		(effects
+			(font
+				(size 1.27 1.27)
+				(color 0 6 255 1)
+			)
+			(justify left)
+		)
+		(property "Intersheetrefs" "${INTERSHEET_REFS}"
+			(at 104.14 55.7978 90)
+			(effects
+				(font
+					(size 1.27 1.27)
+				)
+				(justify left)
+				(hide yes)
+			)
+		)
+	)
 	(global_label "MUX_S3"
 		(shape input)
@@
 		)
 	)
-	(global_label "SENSE2"
+	(global_label "SENSE1"
 		(shape input)
-		(at 386.08 100.33 90)
+		(at 100.33 48.26 90)
 		(fields_autoplaced yes)
 		(effects
 			(font
 				(size 1.27 1.27)
-				(color 255 123 4 1)
+				(color 0 6 255 1)
 			)
 			(justify left)
 		)
 		(property "Intersheetrefs" "${INTERSHEET_REFS}"
-			(at 386.08 90.0878 90)
+			(at 100.33 38.0178 90)
 			(effects
 				(font
@@
 		)
 	)
+	(global_label "SENSE1"
+		(shape input)
+		(at 116.84 30.48 90)
+		(fields_autoplaced yes)
+		(effects
+			(font
+				(size 1.27 1.27)
+				(color 0 6 255 1)
+			)
+			(justify left)
+		)
+		(property "Intersheetrefs" "${INTERSHEET_REFS}"
+			(at 116.84 20.2378 90)
+			(effects
+				(font
+					(size 1.27 1.27)
+				)
+				(justify left)
+				(hide yes)
+			)
+		)
+	)
 	(global_label "MUX3_D10"
 		(shape input)
@@
 			)
 		)
-		(property "Footprint" "FriedSoul_switches:ecs_pad_1U_hybrid_hotswap_V3"
+		(property "Footprint" "FriedSoul_switches:ecs_pad_1U_hybrid_hotswap_V3_switched_sides"
 			(at 196.85 83.82 0)
 			(effects
